File: src/LITEXCNC-HUB75HAT/LITEXCNC-HUB75HAT.kicad_pcb (KiCad board)
At the start: 2 copper layers, 143.5 x 91.4 mm, 63 parts, among them J1 Conn_02x13_Odd_Even, J10 Conn_01x02, J11 HUB75, J12 HUB75, J13 V7.0, J14 V8.0, J15 HUB75, J16 HUB75, J17 Conn_02x20_Odd_Even, J18 Screw_Terminal_01x04, J19 Screw_Terminal_01x04, J2 Conn_02x13_Odd_Even, J3 Conn_02x13_Odd_Even, J4 HUB75, J5 HUB75, J6 HUB75, J7 v7.0, J8 v8.0, J9 HUB75, U1 74CB3T3245, U2 74CB3T3245, U3 74CB3T3245, U4 74CB3T3245, U5 74CB3T3245, U6 74CB3T3245

Commit message: Finished first versiom
Parts:
- removed TP10: TCK, TestPoint:TestPoint_Pad_D1.0mm
- removed TP3, TP4, TP5, TP6: GND, TestPoint:TestPoint_Pad_D1.0mm
- removed TP7: TDO, TestPoint:TestPoint_Pad_D1.0mm
- removed TP8: TDI, TestPoint:TestPoint_Pad_D1.0mm
- removed TP9: TMS, TestPoint:TestPoint_Pad_D1.0mm
- added C10: 33pF, Capacitor_SMD:C_1206_3216Metric_Pad1.33x1.80mm_HandSolder, B.Cu at (208.5, -91.4)
- added C11: 0.1uF, Capacitor_SMD:C_1206_3216Metric_Pad1.33x1.80mm_HandSolder, F.Cu at (199.1, -100.8)
- added C12: 0.1uF, Capacitor_SMD:C_1206_3216Metric_Pad1.33x1.80mm_HandSolder, F.Cu at (207.2, -100.8)
- added C13: 0.1uF, Capacitor_SMD:C_1206_3216Metric_Pad1.33x1.80mm_HandSolder, F.Cu at (198.9, -70.9)
- added C14: 0.1uF, Capacitor_SMD:C_1206_3216Metric_Pad1.33x1.80mm_HandSolder, F.Cu at (206.7, -70.9)
- added C15: 33pF, Capacitor_SMD:C_1206_3216Metric_Pad1.33x1.80mm_HandSolder, B.Cu at (208.3, -61.6)
- added C9: 1nF, Capacitor_SMD:C_1206_3216Metric_Pad1.33x1.80mm_HandSolder, B.Cu at (152.4, -53.0)
- added D1: LED, LED_SMD:LED_1206_3216Metric_Pad1.42x1.75mm_HandSolder, F.Cu at (141.2, -46.7)
- added D10: 1N4148W, Diode_SMD:D_SOD-123, B.Cu at (203.2, -61.5)
- added D11: SM712_SOT23, Package_TO_SOT_SMD:SOT-23, B.Cu at (217.9, -73.2)
- added D12: SM6T6V8A, Diode_SMD:D_SMB, B.Cu at (166.0, -93.0)
- added D2: LED, LED_SMD:LED_1206_3216Metric_Pad1.42x1.75mm_HandSolder, F.Cu at (144.8, -46.7)
- added D3: LED, LED_SMD:LED_1206_3216Metric_Pad1.42x1.75mm_HandSolder, F.Cu at (148.3, -46.7)
- added D4: 1N4148W, Diode_SMD:D_SOD-123, B.Cu at (203.5, -91.3)
- added D5: SM712_SOT23, Package_TO_SOT_SMD:SOT-23, B.Cu at (216.3, -87.4)
- added D6: LED, LED_SMD:LED_1206_3216Metric_Pad1.42x1.75mm_HandSolder, F.Cu at (225.0, -96.0)
- added D7: LED, LED_SMD:LED_1206_3216Metric_Pad1.42x1.75mm_HandSolder, F.Cu at (225.0, -98.6)
- added D8: LED, LED_SMD:LED_1206_3216Metric_Pad1.42x1.75mm_HandSolder, F.Cu at (225.0, -62.7)
- added D9: LED, LED_SMD:LED_1206_3216Metric_Pad1.42x1.75mm_HandSolder, F.Cu at (225.0, -65.3)
- added F1: 108L, Fuse:Fuse_1812_4532Metric_Pad1.30x3.40mm_HandSolder, F.Cu at (217.7, -89.7)
- added F2: 108L, Fuse:Fuse_1812_4532Metric_Pad1.30x3.40mm_HandSolder, F.Cu at (217.7, -85.1)
- added F3: 108L, Fuse:Fuse_1812_4532Metric_Pad1.30x3.40mm_HandSolder, F.Cu at (217.7, -75.4)
- added F4: 108L, Fuse:Fuse_1812_4532Metric_Pad1.30x3.40mm_HandSolder, F.Cu at (217.7, -70.9)
- added F5: 108L, Fuse:Fuse_1812_4532Metric_Pad1.30x3.40mm_HandSolder, F.Cu at (258.8, -63.5)
- added F6: 108L, Fuse:Fuse_1812_4532Metric_Pad1.30x3.40mm_HandSolder, F.Cu at (245.1, -63.5)
- added F7: 108L, Fuse:Fuse_1812_4532Metric_Pad1.30x3.40mm_HandSolder, F.Cu at (230.9, -63.4)
- added R1: 300, Resistor_SMD:R_1206_3216Metric_Pad1.30x1.75mm_HandSolder, F.Cu at (141.2, -54.9)
- added R10: 4.6K, Resistor_SMD:R_1206_3216Metric_Pad1.30x1.75mm_HandSolder, F.Cu at (214.6, -81.8)
- added R11: 120, Resistor_SMD:R_1206_3216Metric_Pad1.30x1.75mm_HandSolder, F.Cu at (213.1, -87.4)
- added R12: 2.4k, Resistor_SMD:R_1206_3216Metric_Pad1.30x1.75mm_HandSolder, F.Cu at (218.7, -96.0)
- added R13: 2.4k, Resistor_SMD:R_1206_3216Metric_Pad1.30x1.75mm_HandSolder, F.Cu at (218.7, -98.6)
- added R14: 2.4k, Resistor_SMD:R_1206_3216Metric_Pad1.30x1.75mm_HandSolder, F.Cu at (218.7, -62.7)
- added R15: 2.4k, Resistor_SMD:R_1206_3216Metric_Pad1.30x1.75mm_HandSolder, F.Cu at (218.7, -65.3)
- added R16: 4.6k, Resistor_SMD:R_1206_3216Metric_Pad1.30x1.75mm_HandSolder, F.Cu at (191.0, -71.0)
- added R17: 56k, Resistor_SMD:R_1206_3216Metric_Pad1.30x1.75mm_HandSolder, B.Cu at (205.7, -61.6)
- added R18: 4.6K, Resistor_SMD:R_1206_3216Metric_Pad1.30x1.75mm_HandSolder, F.Cu at (191.0, -68.5)
- added R19: 4.6K, Resistor_SMD:R_1206_3216Metric_Pad1.30x1.75mm_HandSolder, F.Cu at (214.6, -67.6)
- added R2: 140, Resistor_SMD:R_1206_3216Metric_Pad1.30x1.75mm_HandSolder, F.Cu at (144.8, -54.9)
- added R20: 4.6K, Resistor_SMD:R_1206_3216Metric_Pad1.30x1.75mm_HandSolder, F.Cu at (214.6, -78.7)
- added R21: 120, Resistor_SMD:R_1206_3216Metric_Pad1.30x1.75mm_HandSolder, F.Cu at (213.1, -73.2)
- added R3: 3k3, Resistor_SMD:R_1206_3216Metric_Pad1.30x1.75mm_HandSolder, B.Cu at (150.9, -43.4)
- added R4: 100, Resistor_SMD:R_1206_3216Metric_Pad1.30x1.75mm_HandSolder, B.Cu at (155.2, -53.1)
- added R5: 140, Resistor_SMD:R_1206_3216Metric_Pad1.30x1.75mm_HandSolder, F.Cu at (148.3, -54.9)
- added R6: 4.6k, Resistor_SMD:R_1206_3216Metric_Pad1.30x1.75mm_HandSolder, F.Cu at (191.3, -100.8)
- added R7: 4.6K, Resistor_SMD:R_1206_3216Metric_Pad1.30x1.75mm_HandSolder, F.Cu at (191.3, -98.3)
- added R8: 56k, Resistor_SMD:R_1206_3216Metric_Pad1.30x1.75mm_HandSolder, B.Cu at (206.0, -91.4)
- added R9: 4.6K, Resistor_SMD:R_1206_3216Metric_Pad1.30x1.75mm_HandSolder, F.Cu at (214.6, -93.0)
- added U10: MAX3485, Package_SO:SOIC-8_3.9x4.9mm_P1.27mm, F.Cu at (206.3, -96.6)
- added U11: 74HC04, Package_SO:SOIC-14_3.9x8.7mm_P1.27mm, F.Cu at (197.9, -64.8)
- added U12: MAX3485, Package_SO:SOIC-8_3.9x4.9mm_P1.27mm, F.Cu at (205.7, -66.7)
- added U7: 74HC86, Package_SO:SOIC-14_3.9x8.7mm_P1.27mm, B.Cu at (156.0, -45.5)
- added U8: 74HC02, Package_SO:SOIC-14_3.9x8.7mm_P1.27mm, B.Cu at (164.5, -45.5)
- added U9: 74HC04, Package_SO:SOIC-14_3.9x8.7mm_P1.27mm, F.Cu at (198.2, -94.7)
- J18, J19: value Screw_Terminal_01x04 -> Conn_01x04_Pin; footprint TerminalBlock_Phoenix:TerminalBlock_Phoenix_PTSM-0,5-4-2.5-V-THR_1x04_P2.50mm_Vertical -> Connector_JST:JST_XH_B4B-XH-A_1x04_P2.50mm_Vertical
- moved J19 4.03 mm to (224.5, -69.7)
- moved J18 2.80 mm to (224.5, -83.7)
- moved C3 0.51 mm to (256.2, -69.3)
- moved C5 0.51 mm to (242.2, -69.3)
Connections:
- J1 pad 1: unconnected-(J1-Pin_1-Pad1) -> ENA/ESTOP
- J16 pad 13: unconnected-(J16-Pin_13-Pad13) -> SPI_MISO
- J16 pad 14: unconnected-(J16-Pin_14-Pad14) -> SPI_CLCK
- J16 pad 15: unconnected-(J16-Pin_15-Pad15) -> SPI_MOSI
- J17 pad 10: RXD0 -> RXD1
- J17 pad 32: unconnected-(J17-Pin_32-Pad32) -> TXD5
- J17 pad 33: /JTAG.TCK -> RXD5
- J17 pad 36: unconnected-(J17-Pin_36-Pad36) -> /JTAG.TCK
- J17 pad 8: TXD0 -> TXD1
- J18 pad 1: unconnected-(J18-Pin_1-Pad1) -> GND
- J18 pad 2: unconnected-(J18-Pin_2-Pad2) -> Net-(J18-Pin_2)
- J18 pad 3: unconnected-(J18-Pin_3-Pad3) -> Net-(J18-Pin_3)
- J18 pad 4: unconnected-(J18-Pin_4-Pad4) -> +5V
- J19 pad 1: unconnected-(J19-Pin_1-Pad1) -> GND
- J19 pad 2: unconnected-(J19-Pin_2-Pad2) -> Net-(J19-Pin_2)
- J19 pad 3: unconnected-(J19-Pin_3-Pad3) -> Net-(J19-Pin_3)
- J19 pad 4: unconnected-(J19-Pin_4-Pad4) -> +5V
- J2 pad 1: unconnected-(J2-Pin_1-Pad1) -> ENA/ESTOP
- J3 pad 1: unconnected-(J3-Pin_1-Pad1) -> ENA/ESTOP
- JP1 pad 1: +5V -> Net-(JP1-A)
- JP2 pad 1: +5V -> Net-(JP2-A)
- JP3 pad 1: +5V -> Net-(JP3-A)
Routing:
- net +3.3V: track 176.5 -> 409.9 mm, vias 8 -> 14
- net ENA/ESTOP: track 0.00 -> 202.9 mm, vias 0 -> 1
- net ENA: track 149.9 -> 283.5 mm, vias 4 -> 5
- net TXD5: track 0.00 -> 95.8 mm
- net RXD5: track 0.00 -> 82.7 mm
- net +5V: track 352.3 -> 430.8 mm
- net GND: track 0.00 -> 66.9 mm, vias 8 -> 26
- net Net-(D3-K): track 0.00 -> 39.2 mm, vias 0 -> 1
- net TXD1: track 0.00 -> 39.1 mm
- net Net-(R13-Pad1): track 0.00 -> 29.1 mm, vias 0 -> 2
- net Net-(R12-Pad1): track 0.00 -> 28.4 mm, vias 0 -> 2
- net Net-(R15-Pad1): track 0.00 -> 27.9 mm
- net /JTAG.TMS: track 92.5 -> 66.4 mm
- net Net-(R14-Pad1): track 0.00 -> 25.9 mm
- net Net-(D5-A2): track 0.00 -> 23.5 mm, vias 0 -> 1
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Other:
- board text added: "ENABLE"
- board text added: "ESTOP"
- board text added: "POWER"

Commit message: Proto-type board finished
Parts:
- removed D3: LED, LED_SMD:LED_1206_3216Metric_Pad1.42x1.75mm_HandSolder
- removed U7: 74HC86, Package_SO:SOIC-14_3.9x8.7mm_P1.27mm
- added C16: 0.1uF, Capacitor_SMD:C_1206_3216Metric_Pad1.33x1.80mm_HandSolder, B.Cu at (248.4, -44.2)
- added C17: 0.1uF, Capacitor_SMD:C_1206_3216Metric_Pad1.33x1.80mm_HandSolder, F.Cu at (225.8, -57.1)
- added C18: 0.1uF, Capacitor_SMD:C_1206_3216Metric_Pad1.33x1.80mm_HandSolder, F.Cu at (169.2, -88.1)
- added C19: 0.1uF, Capacitor_SMD:C_1206_3216Metric_Pad1.33x1.80mm_HandSolder, B.Cu at (243.6, -97.0)
- added C20: 0.1uF, Capacitor_SMD:C_1206_3216Metric_Pad1.33x1.80mm_HandSolder, B.Cu at (257.6, -97.0)
- added C21: 0.1uF, Capacitor_SMD:C_1206_3216Metric_Pad1.33x1.80mm_HandSolder, B.Cu at (276.6, -67.3)
- added JP7: SolderJumper_3_Open, Jumper:SolderJumper-3_P2.0mm_Open_TrianglePad1.0x1.5mm, F.Cu at (183.6, -49.8)
- C9: value 1nF -> 0.1uF
- R3: value 3k3 -> R; moved to F.Cu
- R4: value 100 -> R; moved to F.Cu
- R5: value 140 -> R
- U8: value 74HC02 -> 74CB3T3245; footprint Package_SO:SOIC-14_3.9x8.7mm_P1.27mm -> Package_SO:TSSOP-20_4.4x6.5mm_P0.65mm; moved to F.Cu
- moved R3 119.4 mm to (253.7, -104.1), turned to 0 degrees
- moved R4 98.6 mm to (239.5, -104.1), turned to 0 degrees
- moved R5 92.2 mm to (226.5, -103.6), turned to 0 degrees
- moved C9 86.8 mm to (230.1, -91.7), turned to -90 degrees
- moved U8 43.2 mm to (174.0, -87.6), turned to 90 degrees
Connections:
- C9 pad 1: Net-(C9-Pad1) -> +3.3V
- D2 pad 1: Net-(D2-K) -> GND
- J1 pad 1: ENA/ESTOP -> PORTA1
- J16 pad 10: unconnected-(J16-Pin_10-Pad10) -> J4:9
- J16 pad 11: unconnected-(J16-Pin_11-Pad11) -> ENA
- J16 pad 12: unconnected-(J16-Pin_12-Pad12) -> SPI_CS
- J16 pad 8: unconnected-(J16-Pin_8-Pad8) -> J4:7
- J16 pad 9: unconnected-(J16-Pin_9-Pad9) -> J4:8
- J17 pad 24: unconnected-(J17-Pin_24-Pad24) -> SPI_CE0
- J17 pad 26: unconnected-(J17-Pin_26-Pad26) -> SPI_CE1
- J2 pad 1: ENA/ESTOP -> PORTB1
- J3 pad 1: ENA/ESTOP -> PORTC1
- R2 pad 1: +3.3V -> ENA-LED
- R3 pad 1: Net-(R3-Pad1) -> PORTA1
- R3 pad 2: ENA/ESTOP -> Net-(JP4-C)
- R4 pad 1: Net-(C9-Pad1) -> PORTB1
- R4 pad 2: ESTOP -> Net-(JP5-C)
- R5 pad 1: +3.3V -> PORTC1
- R5 pad 2: Net-(D3-A) -> Net-(JP6-C)
- U8 pad 1: Net-(D3-K) -> unconnected-(U8-NC-Pad1)
- U8 pad 10: Net-(U8-Pad10) -> GND
- U8 pad 14: +3.3V -> unconnected-(U8-B4-Pad14)
- U8 pad 2: Net-(U8-Pad10) -> ENA
- U8 pad 3: Net-(U8-Pad3) -> J4:7
- U8 pad 4: Net-(U8-Pad3) -> J4:8
- U8 pad 5: Net-(D3-K) -> J4:9
- U8 pad 6: Net-(R3-Pad1) -> unconnected-(U8-A4-Pad6)
- U8 pad 7: GND -> unconnected-(U8-A5-Pad7)
- U8 pad 8: Net-(U7-Pad11) -> unconnected-(U8-A6-Pad8)
- U8 pad 9: Net-(U7-Pad11) -> unconnected-(U8-A7-Pad9)
Routing:
- net ENA/ESTOP: track 202.9 -> 0.00 mm, vias 1 -> 0
- net PORTA1: track 0.00 -> 112.9 mm
- net PORTB1: track 0.00 -> 97.7 mm
- net PORTC1: track 0.00 -> 82.6 mm
- net J4:9: track 0.00 -> 75.0 mm, vias 0 -> 1
- net J4:8: track 0.00 -> 74.1 mm, vias 0 -> 1
- net J4:7: track 0.00 -> 71.7 mm, vias 0 -> 1
- net ENA-LED: track 0.00 -> 66.1 mm
- net +3.3V: track 409.9 -> 344.6 mm, vias 14 -> 12
- net Net-(D3-K): track 39.2 -> 0.00 mm, vias 1 -> 0
- net ENA: track 283.5 -> 303.8 mm
- net Net-(D2-K): track 20.0 -> 0.00 mm, vias 1 -> 0
- net Net-(R3-Pad1): track 19.9 -> 0.00 mm
- net RXD5: track 82.7 -> 69.0 mm
- net TXD5: track 95.8 -> 82.5 mm
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Other:
- board text added: "CS0"
- board text added: "CS1"
- board text removed: "ESTOP"

Commit message: Prototype ordered
Parts:
- removed J18, J19: Conn_01x04_Pin, Connector_JST:JST_XH_B4B-XH-A_1x04_P2.50mm_Vertical
- added G***: LOGO, LOGO, F.Cu at (158.0, -42.9)
- added RS489-1: Conn_01x02_Pin, Connector_JST:JST_XH_B2B-XH-A_1x02_P2.50mm_Vertical, F.Cu at (225.0, -69.6)
- added RS489-5: Conn_01x02_Pin, Connector_JST:JST_XH_B2B-XH-A_1x02_P2.50mm_Vertical, F.Cu at (225.0, -90.2)
- moved RX 1.02 mm to (225.0, -97.0)
- moved TX 1.02 mm to (225.0, -99.6)
- renumbered D6 to RX, D8 to RX, D9 to TX, D7 to TX
Routing:
- net +5V: track 427.2 -> 401.6 mm
- net Net-(J20-Pin_1): track 4.98 -> 7.16 mm
- net +3.3V: track 344.6 -> 346.6 mm
- net ENA: track 303.8 -> 305.6 mm
- net Net-(J21-Pin_2): track 4.98 -> 6.55 mm
- net Net-(J20-Pin_2): track 5.04 -> 5.90 mm
- net Net-(J21-Pin_1): track 5.03 -> 5.69 mm
- net GND: vias 32 -> 34
Other:
- board text added: "DESIGNED FOR"
- board text added: "HUB75HAT"
- board text added: "V1.0"
