File: src/LITEXCNC-HUB75HAT/LITEXCNC-HUB75HAT.kicad_sch (KiCad schematic)
At the start: 5 parts, among them J14 v7.0, J15 v8.0, J17 Conn_02x20_Odd_Even, J18 Screw_Terminal_01x04, J19 Screw_Terminal_01x04

Commit message: Finished first versiom
Parts:
- removed J18, J19: Screw_Terminal_01x04, TerminalBlock_Phoenix:TerminalBlock_Phoenix_PTSM-0,5-4-2.5-V-THR_1x04_P2.50mm_Vertical, symbol Connector:Screw_Terminal_01x04
- added C9: 1nF, Capacitor_SMD:C_1206_3216Metric_Pad1.33x1.80mm_HandSolder, symbol Device:C
- added D1, D2, D3: LED, LED_SMD:LED_1206_3216Metric_Pad1.42x1.75mm_HandSolder, symbol Device:LED
- added D12: SM6T6V8A, Diode_SMD:D_SMB, symbol Diode:SM6T6V8A
- added R1: 300, Resistor_SMD:R_1206_3216Metric_Pad1.30x1.75mm_HandSolder, symbol Device:R
- added R2, R5: 140, Resistor_SMD:R_1206_3216Metric_Pad1.30x1.75mm_HandSolder, symbol Device:R
- added R3: 3k3, Resistor_SMD:R_1206_3216Metric_Pad1.30x1.75mm_HandSolder, symbol Device:R
- added R4: 100, Resistor_SMD:R_1206_3216Metric_Pad1.30x1.75mm_HandSolder, symbol Device:R
- added U7: 74HC86, Package_SO:SOIC-14_3.9x8.7mm_P1.27mm, symbol 74xx:74HC86
- added U8: 74HC02, Package_SO:SOIC-14_3.9x8.7mm_P1.27mm, symbol 74xx:74HC02
Connections:
- net +3.3V: now also R2.1, R5.1, U7.1, U7.14 (VCC), U7.4, U8.14 (VCC)
- net +5V: now also D12.1 (A1), R1.1
- net GND: now also C9.2, D1.1 (K), D12.2 (A2), U7.7 (GND), U8.7 (GND)
- net JTAG.TCK: now also J17.36 (Pin_36); no longer J17.33 (Pin_33)
- net TXD5: now reaches J17.32 (Pin_32)
- net RXD0 renamed RXD1
- net TXD0 renamed TXD1
- new net: D1.2 (A), R1.2
- new net: D2.2 (A), R2.2
- new net: C9.1, R4.1, U7.13
- new net: U8.10, U8.2
- new net: U7.11, U8.8, U8.9
- new net: D2.1 (K), U7.3, U7.5
- new net: R3.1, U7.6, U7.9, U8.6
- new net: D3.2 (A), R5.2
- new net: D3.1 (K), U8.1, U8.5
- new net: U8.3, U8.4
- new net ENA: U7.2
- new net ENA/ESTOP: R3.2, U7.10
- new net ESTOP: R4.2, U7.12, U7.8
- new net RXD5: J17.33 (Pin_33)
Other:
- added sheet RS485 (schematics/RS485.kicad_sch)
- added sheet RS486 (schematics/RS485.kicad_sch)
- note added: "Status LEDs"

Commit message: Proto-type board finished
Parts:
- removed C9: 1nF, Capacitor_SMD:C_1206_3216Metric_Pad1.33x1.80mm_HandSolder, symbol Device:C
- removed D3: LED, LED_SMD:LED_1206_3216Metric_Pad1.42x1.75mm_HandSolder, symbol Device:LED
- removed R3: 3k3, Resistor_SMD:R_1206_3216Metric_Pad1.30x1.75mm_HandSolder, symbol Device:R
- removed R4: 100, Resistor_SMD:R_1206_3216Metric_Pad1.30x1.75mm_HandSolder, symbol Device:R
- removed R5: 140, Resistor_SMD:R_1206_3216Metric_Pad1.30x1.75mm_HandSolder, symbol Device:R
- removed U7: 74HC86, Package_SO:SOIC-14_3.9x8.7mm_P1.27mm, symbol 74xx:74HC86
- removed U8: 74HC02, Package_SO:SOIC-14_3.9x8.7mm_P1.27mm, symbol 74xx:74HC02
- added JP7: SolderJumper_3_Open, Jumper:SolderJumper-3_P2.0mm_Open_TrianglePad1.0x1.5mm, symbol Jumper:SolderJumper_3_Open
Connections:
- net +3.3V: no longer R2.1
- net GND: now also D2.1 (K)
- net SPI_CE0: now reaches J17.24 (Pin_24)
- net SPI_CE0: now also JP7.1 (A)
- net SPI_CE1: now reaches J17.26 (Pin_26)
- net SPI_CE1: now also JP7.3 (B)
- new net ENA-LED: R2.1
- new net SPI_CS: JP7.2 (C)
Other:
- note added: "Selection of CE signal"
- moved on the sheet: D2, R2

Commit message: Version 1.1
Parts:
- added C5: 100nF, Capacitor_SMD:C_1206_3216Metric_Pad1.33x1.80mm_HandSolder, symbol Device:C_Polarized_Small
- added U7: 74HC04, Package_SO:SOIC-14_3.9x8.7mm_P1.27mm, symbol 74xx:74HC04
- R1: footprint Resistor_SMD:R_1206_3216Metric_Pad1.30x1.75mm_HandSolder -> Resistor_SMD:R_0805_2012Metric_Pad1.20x1.40mm_HandSolder; LCSC (none) -> C17617
- R2: value 140 -> 150; footprint Resistor_SMD:R_1206_3216Metric_Pad1.30x1.75mm_HandSolder -> Resistor_SMD:R_0805_2012Metric_Pad1.20x1.40mm_HandSolder; LCSC (none) -> C17471
Connections:
- net +3.3V: now also C5.1, U7.14 (VCC)
- net ENA-LED: now also U7.6
- net GND: now also C5.2, U7.7 (GND)
- new net: U7.4, U7.5
- new net ENA: U7.2
- new net ENA_IN: U7.1, U7.3
