File: src/daughter_boards/BOB4ENCODER/BOB4ENCODER.kicad_pcb (KiCad board)
At the start: 2 copper layers, 65 x 93 mm, 34 parts, among them J1 Conn_02x13_Odd_Even, J2 Screw_Terminal_01x08, J3 Screw_Terminal_01x08, J4 Screw_Terminal_01x08, J5 Screw_Terminal_01x08, J6 Conn_02x04_Odd_Even, J7 Conn_02x04_Odd_Even, U1 AM26LV32xD, U2 AM26LV32xD, U3 AM26LV32xD

Commit message: Small (non-functional) updates
Parts:
- moved G*** 15.5 mm to (3.05, 53.2)
Routing:
- net GND: track 7.62 -> 83.0 mm, vias 33 -> 52
- net +5V: track 227.3 -> 228.5 mm
- net ENC1_A-: track 97.2 -> 97.6 mm, vias 0 -> 1
- net ENC1_B-: track 106.7 -> 107.1 mm, vias 1 -> 2
- net ENC1_Z-: vias 1 -> 3
