File: src/daughter_boards/BOB4ENCODER/BOB4ENCODER.kicad_sch (KiCad schematic)
At the start: 30 parts, among them J1 Conn_02x13_Odd_Even, J2 Screw_Terminal_01x08, J3 Screw_Terminal_01x08, J4 Screw_Terminal_01x08, J5 Screw_Terminal_01x08, J6 Conn_02x04_Odd_Even, J7 Conn_02x04_Odd_Even, U1 AM26LV32xD, U2 AM26LV32xD, U3 AM26LV32xD

Commit message: Small (non-functional) updates
Parts:
- added D1: MMSZ5222BT1G, Diode_SMD:D_SOD-123, symbol Device:D_Zener
- added R1: R, Resistor_SMD:R_1206_3216Metric_Pad1.30x1.75mm_HandSolder, symbol Device:R
Connections:
- net +5V: now also R1.1
- net GND: now also D1.2 (A)
- net +2V5: now reaches JP4.2 (B), JP5.2 (B), JP6.2 (B)
- net +2V5: now also JP1.2 (B), JP10.2 (B), JP11.2 (B), JP12.2 (B), JP2.2 (B), JP3.2 (B), JP7.2 (B), JP8.2 (B), JP9.2 (B), D1.1 (K), R1.2
Changed lines of the file:
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@@
   (junction (at 269.24 68.58) (diameter 0) (color 0 0 0 0)
+  )
+  (junction (at 129.54 27.94) (diameter 0) (color 0 0 0 0)
   )
   (junction (at 274.32 63.5) (diameter 0) (color 0 0 0 0)
@@
   )
   (wire (pts (xy 46.99 21.59) (xy 46.99 30.48))
+    (stroke (width 0) (type default))
+  )
+  (wire (pts (xy 129.54 27.94) (xy 134.62 27.94))
     (stroke (width 0) (type default))
   )
@@
     (property "Intersheetrefs" "${INTERSHEET_REFS}" (at 27.7178 104.14 0)
       (effects (font (size 1.27 1.27)) (justify right) hide)
+    )
+  )
+  (symbol (lib_id "power:+2V5") (at 96.52 30.48 270) (unit 1)
+    (in_bom yes) (on_board yes) (dnp no) (fields_autoplaced)
+    (property "Reference" "#PWR033" (at 92.71 30.48 0)
+      (effects (font (size 1.27 1.27)) hide)
+    )
+    (property "Value" "+2V5" (at 100.33 30.48 90)
+      (effects (font (size 1.27 1.27)) (justify left))
+    )
+    (property "Footprint" "" (at 96.52 30.48 0)
+      (effects (font (size 1.27 1.27)) hide)
+    )
+    (property "Datasheet" "" (at 96.52 30.48 0)
+      (effects (font (size 1.27 1.27)) hide)
+    )
+    (pin "1")
+    (instances
+      (project "BOB4ENCODER"
+        (path "/9693837c-ee26-4f84-93b4-ccfecde69efc"
+          (reference "#PWR033") (unit 1)
+        )
+      )
     )
   )
@@
     )
   )
+  (symbol (lib_id "power:+2V5") (at 134.62 27.94 270) (unit 1)
+    (in_bom yes) (on_board yes) (dnp no) (fields_autoplaced)
+    (property "Reference" "#PWR034" (at 130.81 27.94 0)
+      (effects (font (size 1.27 1.27)) hide)
+    )
+    (property "Value" "+2V5" (at 138.43 27.94 90)
+      (effects (font (size 1.27 1.27)) (justify left))
+    )
+    (property "Footprint" "" (at 134.62 27.94 0)
+      (effects (font (size 1.27 1.27)) hide)
+    )
+    (property "Datasheet" "" (at 134.62 27.94 0)
+      (effects (font (size 1.27 1.27)) hide)
+    )
+    (pin "1")
+    (instances
+      (project "BOB4ENCODER"
+        (path "/9693837c-ee26-4f84-93b4-ccfecde69efc"
+          (reference "#PWR034") (unit 1)
+        )
+      )
+    )
+  )
   (symbol (lib_id "power:GND") (at 93.98 181.61 0) (unit 1)
     (in_bom yes) (on_board yes) (dnp no) (fields_autoplaced)
@@
         (path "/9693837c-ee26-4f84-93b4-ccfecde69efc"
           (reference "JP5") (unit 1)
+        )
+      )
+    )
+  )
+  (symbol (lib_id "Device:R") (at 129.54 24.13 0) (unit 1)
+    (in_bom yes) (on_board yes) (dnp no) (fields_autoplaced)
+    (property "Reference" "R1" (at 132.08 22.86 0)
+      (effects (font (size 1.27 1.27)) (justify left))
+    )
+    (property "Value" "R" (at 132.08 25.4 0)
+      (effects (font (size 1.27 1.27)) (justify left))
+    )
+    (property "Footprint" "Resistor_SMD:R_1206_3216Metric_Pad1.30x1.75mm_HandSolder" (at 127.762 24.13 90)
+      (effects (font (size 1.27 1.27)) hide)
+    )
+    (property "Datasheet" "~" (at 129.54 24.13 0)
+      (effects (font (size 1.27 1.27)) hide)
+    )
+    (pin "1")
+    (pin "2")
+    (instances
+      (project "BOB4ENCODER"
+        (path "/9693837c-ee26-4f84-93b4-ccfecde69efc"
+          (reference "R1") (unit 1)
         )
       )
@@
     )
   )
+  (symbol (lib_id "power:+2V5") (at 46.99 30.48 270) (unit 1)
+    (in_bom yes) (on_board yes) (dnp no) (fields_autoplaced)
+    (property "Reference" "#PWR030" (at 43.18 30.48 0)
+      (effects (font (size 1.27 1.27)) hide)
+    )
+    (property "Value" "+2V5" (at 50.8 30.48 90)
+      (effects (font (size 1.27 1.27)) (justify left))
+    )
+    (property "Footprint" "" (at 46.99 30.48 0)
+      (effects (font (size 1.27 1.27)) hide)
+    )
+    (property "Datasheet" "" (at 46.99 30.48 0)
+      (effects (font (size 1.27 1.27)) hide)
+    )
+    (pin "1")
+    (instances
+      (project "BOB4ENCODER"
+        (path "/9693837c-ee26-4f84-93b4-ccfecde69efc"
+          (reference "#PWR030") (unit 1)
+        )
+      )
+    )
+  )
   (symbol (lib_id "power:GND") (at 49.53 142.24 0) (unit 1)
     (in_bom yes) (on_board yes) (dnp no) (fields_autoplaced)
@@
         (path "/daea1869-e1ef-4a14-b8f5-612be4c11ee9"
           (reference "#PWR032") (unit 1)
+        )
+      )
+    )
+  )
+  (symbol (lib_id "power:+2V5") (at 46.99 62.23 270) (unit 1)
+    (in_bom yes) (on_board yes) (dnp no) (fields_autoplaced)
+    (property "Reference" "#PWR031" (at 43.18 62.23 0)
+      (effects (font (size 1.27 1.27)) hide)
+    )
+    (property "Value" "+2V5" (at 50.8 62.23 90)
+      (effects (font (size 1.27 1.27)) (justify left))
+    )
+    (property "Footprint" "" (at 46.99 62.23 0)
+      (effects (font (size 1.27 1.27)) hide)
+    )
+    (property "Datasheet" "" (at 46.99 62.23 0)
+      (effects (font (size 1.27 1.27)) hide)
+    )
+    (pin "1")
+    (instances
+      (project "BOB4ENCODER"
+        (path "/9693837c-ee26-4f84-93b4-ccfecde69efc"
+          (reference "#PWR031") (unit 1)
+        )
+      )
+    )
+  )
+  (symbol (lib_id "power:+5V") (at 129.54 20.32 0) (unit 1)
+    (in_bom yes) (on_board yes) (dnp no) (fields_autoplaced)
+    (property "Reference" "#PWR035" (at 129.54 24.13 0)
+      (effects (font (size 1.27 1.27)) hide)
+    )
+    (property "Value" "+5V" (at 129.54 15.24 0)
+      (effects (font (size 1.27 1.27)))
+    )
+    (property "Footprint" "" (at 129.54 20.32 0)
+      (effects (font (size 1.27 1.27)) hide)
+    )
+    (property "Datasheet" "" (at 129.54 20.32 0)
+      (effects (font (size 1.27 1.27)) hide)
+    )
+    (pin "1")
+    (instances
+      (project "BOB4ENCODER"
+        (path "/9693837c-ee26-4f84-93b4-ccfecde69efc"
+          (reference "#PWR035") (unit 1)
+        )
+      )
+      (project "BOB4AXIS"
+        (path "/daea1869-e1ef-4a14-b8f5-612be4c11ee9"
+          (reference "#PWR053") (unit 1)
         )
       )
@@
         (path "/9693837c-ee26-4f84-93b4-ccfecde69efc"
           (reference "JP12") (unit 1)
+        )
+      )
+    )
+  )
+  (symbol (lib_id "Device:D_Zener") (at 129.54 31.75 270) (unit 1)
+    (in_bom yes) (on_board yes) (dnp no) (fields_autoplaced)
+    (property "Reference" "D1" (at 132.08 30.48 90)
+      (effects (font (size 1.27 1.27)) (justify left))
+    )
+    (property "Value" "MMSZ5222BT1G" (at 132.08 33.02 90)
+      (effects (font (size 1.27 1.27)) (justify left))
+    )
+    (property "Footprint" "Diode_SMD:D_SOD-123" (at 129.54 31.75 0)
+      (effects (font (size 1.27 1.27)) hide)
+    )
+    (property "Datasheet" "https://nl.mouser.com/datasheet/2/308/1/MMSZ5221BT1_D-2316205.pdf" (at 129.54 31.75 0)
+      (effects (font (size 1.27 1.27)) hide)
+    )
+    (pin "1")
+    (pin "2")
+    (instances
+      (project "BOB4ENCODER"
+        (path "/9693837c-ee26-4f84-93b4-ccfecde69efc"
+          (reference "D1") (unit 1)
         )
       )
@@
     )
   )
+  (symbol (lib_id "power:GND") (at 129.54 35.56 0) (unit 1)
+    (in_bom yes) (on_board yes) (dnp no) (fields_autoplaced)
+    (property "Reference" "#PWR036" (at 129.54 41.91 0)
+      (effects (font (size 1.27 1.27)) hide)
+    )
+    (property "Value" "GND" (at 129.54 40.64 0)
+      (effects (font (size 1.27 1.27)))
+    )
+    (property "Footprint" "" (at 129.54 35.56 0)
+      (effects (font (size 1.27 1.27)) hide)
+    )
+    (property "Datasheet" "" (at 129.54 35.56 0)
+      (effects (font (size 1.27 1.27)) hide)
+    )
+    (pin "1")
+    (instances
+      (project "BOB4ENCODER"
+        (path "/9693837c-ee26-4f84-93b4-ccfecde69efc"
+          (reference "#PWR036") (unit 1)
+        )
+      )
+      (project "LITEXCNC-HUB75HAT"
+        (path "/d03ad006-987f-4980-aa86-8f7e7030b027/1c7dda94-9358-4abf-bdc6-4f3b8e2b698c"
+          (reference "#PWR015") (unit 1)
+        )
+      )
+      (project "BOB4AXIS"
+        (path "/daea1869-e1ef-4a14-b8f5-612be4c11ee9"
+          (reference "#PWR052") (unit 1)
+        )
+      )
+    )
+  )
   (symbol (lib_id "power:GND") (at 81.28 181.61 0) (unit 1)
     (in_bom yes) (on_board yes) (dnp no) (fields_autoplaced)
@@
         )
       )
+    )
+  )
+  (symbol (lib_id "power:+2V5") (at 96.52 62.23 270) (unit 1)
+    (in_bom yes) (on_board yes) (dnp no) (fields_autoplaced)
+    (property "Reference" "#PWR032" (at 92.71 62.23 0)
+      (effects (font (size 1.27 1.27)) hide)
+    )
+    (property "Value" "+2V5" (at 100.33 62.23 90)
+      (effects (font (size 1.27 1.27)) (justify left))
+    )
+    (property "Footprint" "" (at 96.52 62.23 0)
+      (effects (font (size 1.27 1.27)) hide)
+    )
+    (property "Datasheet" "" (at 96.52 62.23 0)
+      (effects (font (size 1.27 1.27)) hide)
+    )
+    (pin "1")
+    (instances
+      (project "BOB4ENCODER"
+        (path "/9693837c-ee26-4f84-93b4-ccfecde69efc"
+          (reference "#PWR032") (unit 1)
+        )
+      )
