File: src/LITEXCNC-HUB75HAT/schematics/IO.kicad_sch (KiCad schematic)
At the start: 27 parts, among them J1 Conn_02x13_Odd_Even, J2 Conn_02x13_Odd_Even, J3 Conn_02x13_Odd_Even

Commit message: Finished first versiom
Parts:
- added F1 (x3): 108L, Fuse:Fuse_1812_4532Metric_Pad1.30x3.40mm_HandSolder, symbol Device:Polyfuse
Connections:
- net +5V: now also F1.1, F1.1, F1.1; no longer JP1.1 (A), JP2.1 (A), JP3.1 (A)
- net ENA/ESTOP: now reaches J2.1 (Pin_1)
- net ENA/ESTOP: now also J1.1 (Pin_1), J3.1 (Pin_1)
- new net: F1.2, JP2.1 (A)
- new net: F1.2, JP3.1 (A)
- new net: F1.2, JP1.1 (A)

Commit message: Proto-type board finished
Parts:
- added R3, R4, R5: R, Resistor_SMD:R_1206_3216Metric_Pad1.30x1.75mm_HandSolder, symbol Device:R
Connections:
- net at JP5.2 (C), RN5.1 (R1.1), RN5.2 (R2.1)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: now also R4.2
- net at JP4.2 (C), RN1.1 (R1.1), RN1.2 (R2.1)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: now also R3.2
- net at JP6.2 (C), RN10.1 (R1.1), RN10.2 (R2.1)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: now also R5.2
- removed net ENA/ESTOP: J1.1 (Pin_1), J2.1 (Pin_1), J3.1 (Pin_1)
- new net PORTA1: J1.1 (Pin_1), R3.1
- new net PORTB1: J2.1 (Pin_1), R4.1
- new net PORTC1: J3.1 (Pin_1), R5.1
Changed lines of the file:
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@@
   (junction (at 85.09 130.81) (diameter 0) (color 0 0 0 0)
   )
+  (junction (at 38.1 148.59) (diameter 0) (color 0 0 0 0)
+  )
   (junction (at 107.95 43.18) (diameter 0) (color 0 0 0 0)
   )
@@
   (junction (at 220.98 83.82) (diameter 0) (color 0 0 0 0)
   )
+  (junction (at 85.09 148.59) (diameter 0) (color 0 0 0 0)
+  )
   (junction (at 69.85 43.18) (diameter 0) (color 0 0 0 0)
   )
@@
   (junction (at 85.09 128.27) (diameter 0) (color 0 0 0 0)
   )
+  (junction (at 133.35 148.59) (diameter 0) (color 0 0 0 0)
+  )
   (junction (at 85.09 92.71) (diameter 0) (color 0 0 0 0)
   )
@@
     (stroke (width 0) (type default))
   )
+  (wire (pts (xy 133.35 148.59) (xy 133.35 157.48))
+    (stroke (width 0) (type default))
+  )
   (wire (pts (xy 60.96 38.1) (xy 69.85 38.1))
     (stroke (width 0) (type default))
@@
     (stroke (width 0) (type default))
   )
+  (wire (pts (xy 85.09 148.59) (xy 85.09 157.48))
+    (stroke (width 0) (type default))
+  )
   (wire (pts (xy 137.16 38.1) (xy 146.05 38.1))
     (stroke (width 0) (type default))
@@
     (stroke (width 0) (type default))
   )
+  (wire (pts (xy 86.36 157.48) (xy 85.09 157.48))
+    (stroke (width 0) (type default))
+  )
   (wire (pts (xy 133.35 95.25) (xy 133.35 105.41))
     (stroke (width 0) (type default))
   )
+  (wire (pts (xy 38.1 148.59) (xy 38.1 157.48))
+    (stroke (width 0) (type default))
+  )
   (wire (pts (xy 133.35 105.41) (xy 133.35 107.95))
     (stroke (width 0) (type default))
@@
     (stroke (width 0) (type default))
   )
+  (wire (pts (xy 134.62 157.48) (xy 133.35 157.48))
+    (stroke (width 0) (type default))
+  )
   (wire (pts (xy 107.95 43.18) (xy 107.95 45.72))
     (stroke (width 0) (type default))
@@
     (stroke (width 0) (type default))
   )
+  (wire (pts (xy 39.37 157.48) (xy 38.1 157.48))
+    (stroke (width 0) (type default))
+  )
   (wire (pts (xy 38.1 125.73) (xy 38.1 128.27))
     (stroke (width 0) (type default))
@@
     )
   )
+  (global_label "PORTA1" (shape bidirectional) (at 46.99 157.48 0) (fields_autoplaced)
+    (effects (font (size 1.1 1.1)) (justify left))
+    (property "Intersheetrefs" "${INTERSHEET_REFS}" (at 56.7188 157.48 0)
+      (effects (font (size 1.27 1.27)) (justify left) hide)
+    )
+  )
   (global_label "PORTC15" (shape bidirectional) (at 137.16 30.48 0) (fields_autoplaced)
     (effects (font (size 1.1 1.1)) (justify left))
@@
     )
   )
+  (global_label "PORTA1" (shape bidirectional) (at 48.26 27.94 180) (fields_autoplaced)
+    (effects (font (size 1.1 1.1)) (justify right))
+    (property "Intersheetrefs" "${INTERSHEET_REFS}" (at 38.5312 27.94 0)
+      (effects (font (size 1.27 1.27)) (justify right) hide)
+    )
+  )
   (global_label "PORTC8" (shape bidirectional) (at 124.46 45.72 180) (fields_autoplaced)
     (effects (font (size 1.1 1.1)) (justify right))
     (property "Intersheetrefs" "${INTERSHEET_REFS}" (at 114.5741 45.72 0)
-      (effects (font (size 1.27 1.27)) (justify right) hide)
-    )
-  )
-  (global_label "ENA{slash}ESTOP" (shape bidirectional) (at 86.36 27.94 180) (fields_autoplaced)
-    (effects (font (size 1.1 1.1)) (justify right))
-    (property "Intersheetrefs" "${INTERSHEET_REFS}" (at 73.436 27.94 0)
       (effects (font (size 1.27 1.27)) (justify right) hide)
     )
@@
     )
   )
+  (global_label "PORTB1" (shape bidirectional) (at 86.36 27.94 180) (fields_autoplaced)
+    (effects (font (size 1.1 1.1)) (justify right))
+    (property "Intersheetrefs" "${INTERSHEET_REFS}" (at 76.4741 27.94 0)
+      (effects (font (size 1.27 1.27)) (justify right) hide)
+    )
+  )
   (global_label "PORTB6" (shape bidirectional) (at 86.36 40.64 180) (fields_autoplaced)
     (effects (font (size 1.1 1.1)) (justify right))
@@
     )
   )
-  (global_label "ENA{slash}ESTOP" (shape bidirectional) (at 124.46 27.94 180) (fields_autoplaced)
-    (effects (font (size 1.1 1.1)) (justify right))
-    (property "Intersheetrefs" "${INTERSHEET_REFS}" (at 111.536 27.94 0)
+  (global_label "PORTC1" (shape bidirectional) (at 124.46 27.94 180) (fields_autoplaced)
+    (effects (font (size 1.1 1.1)) (justify right))
+    (property "Intersheetrefs" "${INTERSHEET_REFS}" (at 114.5741 27.94 0)
       (effects (font (size 1.27 1.27)) (justify right) hide)
     )
@@
     )
   )
-  (global_label "ENA{slash}ESTOP" (shape bidirectional) (at 48.26 27.94 180) (fields_autoplaced)
-    (effects (font (size 1.1 1.1)) (justify right))
-    (property "Intersheetrefs" "${INTERSHEET_REFS}" (at 35.336 27.94 0)
-      (effects (font (size 1.27 1.27)) (justify right) hide)
+  (global_label "PORTB1" (shape bidirectional) (at 93.98 157.48 0) (fields_autoplaced)
+    (effects (font (size 1.1 1.1)) (justify left))
+    (property "Intersheetrefs" "${INTERSHEET_REFS}" (at 103.8659 157.48 0)
+      (effects (font (size 1.27 1.27)) (justify left) hide)
     )
   )
@@
     (effects (font (size 1.1 1.1)) (justify left))
     (property "Intersheetrefs" "${INTERSHEET_REFS}" (at 105.1359 92.71 0)
+      (effects (font (size 1.27 1.27)) (justify left) hide)
+    )
+  )
+  (global_label "PORTC1" (shape bidirectional) (at 142.24 157.48 0) (fields_autoplaced)
+    (effects (font (size 1.1 1.1)) (justify left))
+    (property "Intersheetrefs" "${INTERSHEET_REFS}" (at 152.1259 157.48 0)
       (effects (font (size 1.27 1.27)) (justify left) hide)
     )
@@
         (path "/d03ad006-987f-4980-aa86-8f7e7030b027/1c7dda94-9358-4abf-bdc6-4f3b8e2b698c"
           (reference "#PWR022") (unit 1)
+        )
+      )
+    )
+  )
+  (symbol (lib_id "Device:R") (at 138.43 157.48 270) (unit 1)
+    (in_bom yes) (on_board yes) (dnp no) (fields_autoplaced)
+    (property "Reference" "R5" (at 138.43 151.13 90)
+      (effects (font (size 1.27 1.27)))
+    )
+    (property "Value" "R" (at 138.43 153.67 90)
+      (effects (font (size 1.27 1.27)))
+    )
+    (property "Footprint" "Resistor_SMD:R_1206_3216Metric_Pad1.30x1.75mm_HandSolder" (at 138.43 155.702 90)
+      (effects (font (size 1.27 1.27)) hide)
+    )
+    (property "Datasheet" "~" (at 138.43 157.48 0)
+      (effects (font (size 1.27 1.27)) hide)
+    )
+    (pin "1")
+    (pin "2")
+    (instances
+      (project "LITEXCNC-HUB75HAT"
+        (path "/d03ad006-987f-4980-aa86-8f7e7030b027/1c7dda94-9358-4abf-bdc6-4f3b8e2b698c"
+          (reference "R5") (unit 1)
         )
       )
@@
         )
       )
+    )
+  )
+  (symbol (lib_id "Device:R") (at 90.17 157.48 270) (unit 1)
+    (in_bom yes) (on_board yes) (dnp no) (fields_autoplaced)
+    (property "Reference" "R4" (at 90.17 151.13 90)
+      (effects (font (size 1.27 1.27)))
+    )
+    (property "Value" "R" (at 90.17 153.67 90)
+      (effects (font (size 1.27 1.27)))
+    )
+    (property "Footprint" "Resistor_SMD:R_1206_3216Metric_Pad1.30x1.75mm_HandSolder" (at 90.17 155.702 90)
+      (effects (font (size 1.27 1.27)) hide)
+    )
+    (property "Datasheet" "~" (at 90.17 157.48 0)
+      (effects (font (size 1.27 1.27)) hide)
+    )
+    (pin "1")
+    (pin "2")
+    (instances
+      (project "LITEXCNC-HUB75HAT"
+        (path "/d03ad006-987f-4980-aa86-8f7e7030b027/1c7dda94-9358-4abf-bdc6-4f3b8e2b698c"
+          (reference "R4") (unit 1)
+        )
+      )
+    )
+  )
+  (symbol (lib_id "Device:R") (at 43.18 157.48 270) (unit 1)
+    (in_bom yes) (on_board yes) (dnp no) (fields_autoplaced)
+    (property "Reference" "R3" (at 43.18 151.13 90)
+      (effects (font (size 1.27 1.27)))
+    )
+    (property "Value" "R" (at 43.18 153.67 90)
+      (effects (font (size 1.27 1.27)))
+    )
+    (property "Footprint" "Resistor_SMD:R_1206_3216Metric_Pad1.30x1.75mm_HandSolder" (at 43.18 155.702 90)
+      (effects (font (size 1.27 1.27)) hide)
+    )
+    (property "Datasheet" "~" (at 43.18 157.48 0)
+      (effects (font (size 1.27 1.27)) hide)
+    )
+    (pin "1")
+    (pin "2")
+    (instances
+      (project "LITEXCNC-HUB75HAT"
+        (path "/d03ad006-987f-4980-aa86-8f7e7030b027/1c7dda94-9358-4abf-bdc6-4f3b8e2b698c"
+          (reference "R3") (unit 1)
+        )
+      )

Commit message: Version 1.1
Parts:
- C1, C2, C3, C4, C5, C6: value 0.1uF -> 100nF; LCSC (none) -> C24497
- F1: LCSC (none) -> C782760
- J1, J2, J3: footprint Connector_PinHeader_2.54mm:PinHeader_2x13_P2.54mm_Vertical -> Connector_IDC:IDC-Header_2x13_P2.54mm_Vertical
- R3, R4, R5: LCSC (none) -> C17902
- RN1, RN10, RN11, RN12, RN2, RN3, RN4, RN5, RN6, RN7, RN8, RN9: value 3.3k -> CN1J4KTTD1002F; footprint Resistor_SMD:R_Array_Convex_4x1206 -> Resistor_SMD:R_Array_Convex_4x0603_handsolder; LCSC (none) -> C29718
