File: src/LITEXCNC-HUB75HAT/schematics/RS485.kicad_sch (KiCad schematic)
At the start: 20 parts, among them J18 Conn_01x04_Pin, U10 MAX3485, U9 74HC04

Commit message: Prototype ordered
Parts:
- removed J18: Conn_01x04_Pin, Connector_JST:JST_XH_B4B-XH-A_1x04_P2.50mm_Vertical, symbol Connector:Conn_01x04_Pin
- added J20: Conn_01x02_Pin, symbol Connector:Conn_01x02_Pin
Connections:
- net at F2.1: now also J20.1 (Pin_1)
- net at F1.2: now also J20.2 (Pin_2)
Changed lines of the file:
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@@
-    )
-  )
-  (symbol (lib_id "Connector:Conn_01x04_Pin") (at 250.19 54.61 180) (unit 1)
-    (in_bom yes) (on_board yes) (dnp no)
-    (property "Reference" "J18" (at 249.555 62.23 0)
-      (effects (font (size 1.27 1.27)))
-    )
-    (property "Value" "Conn_01x04_Pin" (at 249.555 59.69 0)
-      (effects (font (size 1.27 1.27)))
-    )
-    (property "Footprint" "Connector_JST:JST_XH_B4B-XH-A_1x04_P2.50mm_Vertical" (at 250.19 54.61 0)
-      (effects (font (size 1.27 1.27)) hide)
-    )
-    (property "Datasheet" "~" (at 250.19 54.61 0)
-      (effects (font (size 1.27 1.27)) hide)
-    )
-    (pin "1")
-    (pin "2")
-    (pin "3")
-    (pin "4")
-    (instances
-      (project "LITEXCNC-HUB75HAT"
-        (path "/d03ad006-987f-4980-aa86-8f7e7030b027"
-          (reference "J18") (unit 1)
-        )
-        (path "/d03ad006-987f-4980-aa86-8f7e7030b027/7e4767b4-b2d0-42d7-8d39-43025a744821"
-          (reference "J18") (unit 1)
-        )
-        (path "/d03ad006-987f-4980-aa86-8f7e7030b027/9bb13272-be2a-4c45-a57a-353180fffd14"
-          (reference "J19") (unit 1)
-        )
-      )
     )
   )
@@
     )
   )
+  (symbol (lib_id "Connector:Conn_01x02_Pin") (at 250.19 54.61 180) (unit 1)
+    (in_bom yes) (on_board yes) (dnp no) (fields_autoplaced)
+    (property "Reference" "J20" (at 251.46 52.07 0)
+      (effects (font (size 1.27 1.27)) (justify right))
+    )
+    (property "Value" "Conn_01x02_Pin" (at 251.46 54.61 0)
+      (effects (font (size 1.27 1.27)) (justify right))
+    )
+    (property "Footprint" "" (at 250.19 54.61 0)
+      (effects (font (size 1.27 1.27)) hide)
+    )
+    (property "Datasheet" "~" (at 250.19 54.61 0)
+      (effects (font (size 1.27 1.27)) hide)
+    )
+    (pin "1")
+    (pin "2")
+    (instances
+      (project "LITEXCNC-HUB75HAT"
+        (path "/d03ad006-987f-4980-aa86-8f7e7030b027/7e4767b4-b2d0-42d7-8d39-43025a744821"
+          (reference "J20") (unit 1)
+        )
+        (path "/d03ad006-987f-4980-aa86-8f7e7030b027/9bb13272-be2a-4c45-a57a-353180fffd14"
+          (reference "J21") (unit 1)
+        )
+      )
+    )
+  )
   (symbol (lib_id "74xx:74HC04") (at 91.44 66.04 0) (unit 5)
     (in_bom yes) (on_board yes) (dnp no) (fields_autoplaced)
@@
     )
   )
-  (symbol (lib_id "power:+5V") (at 245.11 49.53 90) (unit 1)
-    (in_bom yes) (on_board yes) (dnp no) (fields_autoplaced)
-    (property "Reference" "#PWR0104" (at 248.92 49.53 0)
-      (effects (font (size 1.27 1.27)) hide)
-    )
-    (property "Value" "+5V" (at 241.3 49.53 90)
-      (effects (font (size 1.27 1.27)) (justify left))
-    )
-    (property "Footprint" "" (at 245.11 49.53 0)
-      (effects (font (size 1.27 1.27)) hide)
-    )
-    (property "Datasheet" "" (at 245.11 49.53 0)
-      (effects (font (size 1.27 1.27)) hide)
-    )
-    (pin "1")
-    (instances
-      (project "LITEXCNC-HUB75HAT"
-        (path "/d03ad006-987f-4980-aa86-8f7e7030b027/7e4767b4-b2d0-42d7-8d39-43025a744821"
-          (reference "#PWR0104") (unit 1)
-        )
-        (path "/d03ad006-987f-4980-aa86-8f7e7030b027/9bb13272-be2a-4c45-a57a-353180fffd14"
-          (reference "#PWR0105") (unit 1)
-        )
-      )
-    )
-  )
   (symbol (lib_id "Device:R") (at 102.87 25.4 90) (unit 1)
     (in_bom yes) (on_board yes) (dnp no) (fields_autoplaced)
@@
         )
       )
-    )
-  )
-  (symbol (lib_id "power:GND") (at 245.11 57.15 270) (unit 1)
-    (in_bom yes) (on_board yes) (dnp no) (fields_autoplaced)
-    (property "Reference" "#PWR0102" (at 238.76 57.15 0)
-      (effects (font (size 1.27 1.27)) hide)
-    )
-    (property "Value" "GND" (at 241.3 57.15 90)
-      (effects (font (size 1.27 1.27)) (justify right))
-    )
-    (property "Footprint" "" (at 245.11 57.15 0)
-      (effects (font (size 1.27 1.27)) hide)
-    )
-    (property "Datasheet" "" (at 245.11 57.15 0)
-      (effects (font (size 1.27 1.27)) hide)
-    )
-    (pin "1")
-    (instances
-      (project "LITEXCNC-HUB75HAT"
-        (path "/d03ad006-987f-4980-aa86-8f7e7030b027/7e4767b4-b2d0-42d7-8d39-43025a744821"
-          (reference "#PWR0102") (unit 1)
-        )
-        (path "/d03ad006-987f-4980-aa86-8f7e7030b027/9bb13272-be2a-4c45-a57a-353180fffd14"
-          (reference "#PWR0103") (unit 1)
-        )
-      )

Commit message: Version 1.1
Parts:
- C10: footprint Capacitor_SMD:C_1206_3216Metric_Pad1.33x1.80mm_HandSolder -> Capacitor_SMD:C_0603_1608Metric_Pad1.08x0.95mm_HandSolder; LCSC (none) -> C1663
- C11: value 0.1uF -> 100nF; LCSC (none) -> C24497
- C12: LCSC (none) -> C24497
- D5: LCSC (none) -> C2687124
- F1, F2: LCSC (none) -> C782760
- R10, R7, R9: value 4.6K -> 4.7K; LCSC (none) -> C17936
- R11: LCSC (none) -> C17909
- R12, R13: value 2.4k -> 150; footprint Resistor_SMD:R_1206_3216Metric_Pad1.30x1.75mm_HandSolder -> Resistor_SMD:R_0805_2012Metric_Pad1.20x1.40mm_HandSolder; LCSC (none) -> C17471
- R6: value 4.6k -> 4.7k; LCSC (none) -> C17936
- R8: footprint Resistor_SMD:R_1206_3216Metric_Pad1.30x1.75mm_HandSolder -> Resistor_SMD:R_0603_1608Metric_Pad0.98x0.95mm_HandSolder; LCSC (none) -> C23206
- U10: LCSC (none) -> C8963
Changed lines of the file:
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@@
       (effects (font (size 1.27 1.27)) (justify left))
     )
-    (property "Value" "4.6k" (at 80.01 63.5 0)
+    (property "Value" "4.7k" (at 80.01 63.5 0)
       (effects (font (size 1.27 1.27)) (justify left))
     )
@@
       (effects (font (size 1.27 1.27)) hide)
     )
+    (property "LCSC" "C17936" (at 77.47 62.23 0)
+      (effects (font (size 1.27 1.27)) hide)
+    )
     (pin "1")
     (pin "2")
@@
       (effects (font (size 1.27 1.27)) (justify left))
     )
-    (property "Value" "4.6K" (at 181.61 64.77 0)
+    (property "Value" "4.7K" (at 181.61 64.77 0)
       (effects (font (size 1.27 1.27)) (justify left))
     )
@@
     )
     (property "Datasheet" "~" (at 179.07 63.5 0)
+      (effects (font (size 1.27 1.27)) hide)
+    )
+    (property "LCSC" "C17936" (at 179.07 63.5 0)
       (effects (font (size 1.27 1.27)) hide)
     )
@@
     )
     (property "Datasheet" "https://www.littelfuse.com/~/media/electronics/datasheets/tvs_diode_arrays/littelfuse_tvs_diode_array_sm712_datasheet.pdf.pdf" (at 210.82 50.8 0)
+      (effects (font (size 1.27 1.27)) hide)
+    )
+    (property "LCSC" "C2687124" (at 210.82 54.61 90)
       (effects (font (size 1.27 1.27)) hide)
     )
@@
       (effects (font (size 1.27 1.27)) hide)
     )
+    (property "LCSC" "C782760" (at 226.06 45.72 90)
+      (effects (font (size 1.27 1.27)) hide)
+    )
     (pin "1")
     (pin "2")
@@
       (effects (font (size 1.27 1.27)))
     )
-    (property "Value" "2.4k" (at 102.87 21.59 90)
-      (effects (font (size 1.27 1.27)))
-    )
-    (property "Footprint" "Resistor_SMD:R_1206_3216Metric_Pad1.30x1.75mm_HandSolder" (at 102.87 27.178 90)
+    (property "Value" "150" (at 102.87 21.59 90)
+      (effects (font (size 1.27 1.27)))
+    )
+    (property "Footprint" "Resistor_SMD:R_0805_2012Metric_Pad1.20x1.40mm_HandSolder" (at 102.87 27.178 90)
       (effects (font (size 1.27 1.27)) hide)
     )
@@
       (effects (font (size 1.27 1.27)) hide)
     )
+    (property "LCSC" "C17471" (at 102.87 25.4 90)
+      (effects (font (size 1.27 1.27)) hide)
+    )
     (pin "1")
     (pin "2")
@@
       (effects (font (size 1.27 1.27)) (justify left))
     )
-    (property "Footprint" "Capacitor_SMD:C_1206_3216Metric_Pad1.33x1.80mm_HandSolder" (at 135.5852 82.55 0)
+    (property "Footprint" "Capacitor_SMD:C_0603_1608Metric_Pad1.08x0.95mm_HandSolder" (at 135.5852 82.55 0)
       (effects (font (size 1.27 1.27)) hide)
     )
     (property "Datasheet" "~" (at 134.62 78.74 0)
+      (effects (font (size 1.27 1.27)) hide)
+    )
+    (property "LCSC" "C1663" (at 134.62 78.74 0)
       (effects (font (size 1.27 1.27)) hide)
     )
@@
       (effects (font (size 1.27 1.27)) hide)
     )
+    (property "LCSC" "C17909" (at 186.69 54.61 0)
+      (effects (font (size 1.27 1.27)) hide)
+    )
     (pin "1")
     (pin "2")
@@
     )
     (property "Datasheet" "~" (at 226.06 63.5 0)
+      (effects (font (size 1.27 1.27)) hide)
+    )
+    (property "LCSC" "C782760" (at 226.06 63.5 90)
       (effects (font (size 1.27 1.27)) hide)
     )
@@
       (effects (font (size 1.27 1.27)) hide)
     )
+    (property "LCSC" "C24497" (at 72.39 186.69 0)
+      (effects (font (size 1.27 1.27)) hide)
+    )
     (pin "1")
     (pin "2")
@@
     )
     (property "Datasheet" "https://datasheets.maximintegrated.com/en/ds/MAX3483-MAX3491.pdf" (at 160.02 52.07 0)
+      (effects (font (size 1.27 1.27)) hide)
+    )
+    (property "LCSC" "C8963" (at 160.02 53.34 0)
       (effects (font (size 1.27 1.27)) hide)
     )
@@
       (effects (font (size 1.27 1.27)) (justify left))
     )
-    (property "Value" "4.6K" (at 177.8 45.72 0)
+    (property "Value" "4.7K" (at 177.8 45.72 0)
       (effects (font (size 1.27 1.27)) (justify left))
     )
@@
     )
     (property "Datasheet" "~" (at 175.26 44.45 0)
+      (effects (font (size 1.27 1.27)) hide)
+    )
+    (property "LCSC" "C17936" (at 175.26 44.45 0)
       (effects (font (size 1.27 1.27)) hide)
     )
@@
       (effects (font (size 1.27 1.27)) (justify left))
     )
-    (property "Value" "4.6K" (at 152.4 38.1 0)
+    (property "Value" "4.7K" (at 152.4 38.1 0)
       (effects (font (size 1.27 1.27)) (justify left))
     )
@@
     )
     (property "Datasheet" "~" (at 149.86 36.83 0)
+      (effects (font (size 1.27 1.27)) hide)
+    )
+    (property "LCSC" "C17936" (at 149.86 36.83 0)
       (effects (font (size 1.27 1.27)) hide)
     )
@@
       (effects (font (size 1.27 1.27)) (justify left))
     )
-    (property "Value" "0.1uF" (at 59.69 187.96 0)
+    (property "Value" "100nF" (at 59.69 187.96 0)
       (effects (font (size 1.27 1.27)) (justify left))
     )
@@
       (effects (font (size 1.27 1.27)) hide)
     )
+    (property "LCSC" "C24497" (at 55.88 186.69 0)
+      (effects (font (size 1.27 1.27)) hide)
+    )
     (pin "1")
     (pin "2")
@@
       (effects (font (size 1.27 1.27)))
     )
-    (property "Value" "2.4k" (at 102.87 73.66 90)
-      (effects (font (size 1.27 1.27)))
-    )
-    (property "Footprint" "Resistor_SMD:R_1206_3216Metric_Pad1.30x1.75mm_HandSolder" (at 97.282 73.66 90)
+    (property "Value" "150" (at 102.87 73.66 90)
+      (effects (font (size 1.27 1.27)))
+    )
+    (property "Footprint" "Resistor_SMD:R_0805_2012Metric_Pad1.20x1.40mm_HandSolder" (at 97.282 73.66 90)
       (effects (font (size 1.27 1.27)) hide)
     )
     (property "Datasheet" "~" (at 99.06 73.66 0)
+      (effects (font (size 1.27 1.27)) hide)
+    )
+    (property "LCSC" "C17471" (at 99.06 73.66 90)
       (effects (font (size 1.27 1.27)) hide)
     )
@@
       (effects (font (size 1.27 1.27)))
     )
-    (property "Footprint" "Resistor_SMD:R_1206_3216Metric_Pad1.30x1.75mm_HandSolder" (at 130.81 72.898 90)
+    (property "Footprint" "Resistor_SMD:R_0603_1608Metric_Pad0.98x0.95mm_HandSolder" (at 130.81 72.898 90)
       (effects (font (size 1.27 1.27)) hide)
     )
@@
       (effects (font (size 1.27 1.27)) hide)
     )
+    (property "LCSC" "C23206" (at 130.81 71.12 90)
+      (effects (font (size 1.27 1.27)) hide)
+    )
