File: src/LITEXCNC-HUB75HAT/schematics/buffers.kicad_sch (KiCad schematic)
At the start: 6 parts, among them U1 74CB3T3245, U2 74CB3T3245, U3 74CB3T3245, U4 74CB3T3245, U5 74CB3T3245, U6 74CB3T3245

Commit message: Proto-type board finished
Parts:
- added C5 (x7): 0.1uF, Capacitor_SMD:C_1206_3216Metric_Pad1.33x1.80mm_HandSolder, symbol Device:C_Polarized_Small
- added U8: 74CB3T3245, Package_SO:TSSOP-20_4.4x6.5mm_P0.65mm, symbol Custom_components:74CB3T3245
Connections:
- net +3.3V: now also C5.1, C5.1, C5.1, C5.1, C5.1, C5.1, C5.1, U8.20 (VCC)
- net ENA: now also U8.19 (CE), U8.2 (A0)
- net GND: now also C5.2, C5.2, C5.2, C5.2, C5.2, C5.2, C5.2, U8.10 (GND)
- new net ENA-LED: U8.18 (B0)
- new net J4:7: U8.3 (A1)
- new net J4:8: U8.4 (A2)
- new net J4:9: U8.5 (A3)
- new net PORTA1: U8.17 (B1)
- new net PORTB1: U8.16 (B2)
- new net PORTC1: U8.15 (B3)

Commit message: Version 1.1
Parts:
- C5: value 0.1uF -> 100nF; LCSC (none) -> C24497
- U1, U2, U3, U4, U5, U6, U8: LCSC (none) -> C15298
Connections:
- net ENA: no longer U8.2 (A0)
- net J4:7: now also U8.9 (A7); no longer U8.3 (A1)
- net J4:8: now also U8.8 (A6); no longer U8.4 (A2)
- net J4:9: now also U8.7 (A5); no longer U8.5 (A3)
- net PORTA1: now also U8.11 (B7); no longer U8.17 (B1)
- net PORTB1: now also U8.12 (B6); no longer U8.16 (B2)
- net PORTC1: now also U8.13 (B5); no longer U8.15 (B3)
- net ENA-LED: no longer names the net of U8.18 (B0)
