File: src/LITEXCNC-HUB75HAT/schematics/hub75.kicad_sch (KiCad schematic)
At the start: 13 parts, among them J11 HUB75, J12 HUB75, J13 HUB75, J16 HUB75, J17 Conn_01x02, J18 HUB75, J19 HUB75, J20 V7.0, J21 V8.0, J22 HUB75, J23 HUB75

Commit message: Finished first versiom
Connections:
- net SPI_MISO: now reaches J23.13 (Pin_13)
- net SPI_CLCK: now reaches J23.14 (Pin_14)
- net SPI_MOSI: now reaches J23.15 (Pin_15)
Changed lines of the file:
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@@
+    )
+  )
+  (global_label "SPI_MISO" (shape output) (at 49.53 80.01 270) (fields_autoplaced)
+    (effects (font (size 1 1)) (justify right))
+    (property "Intersheetrefs" "${INTERSHEET_REFS}" (at 49.53 89.1699 90)
+      (effects (font (size 1.27 1.27)) (justify right) hide)
     )
   )
@@
     )
   )
+  (global_label "SPI_CLCK" (shape input) (at 49.53 67.31 90) (fields_autoplaced)
+    (effects (font (size 1 1)) (justify left))
+    (property "Intersheetrefs" "${INTERSHEET_REFS}" (at 49.53 57.9597 90)
+      (effects (font (size 1.27 1.27)) (justify left) hide)
+    )
+  )
+  (global_label "SPI_MOSI" (shape input) (at 52.07 80.01 270) (fields_autoplaced)
+    (effects (font (size 1 1)) (justify right))
+    (property "Intersheetrefs" "${INTERSHEET_REFS}" (at 52.07 89.1699 90)
+      (effects (font (size 1.27 1.27)) (justify right) hide)
+    )
+  )
   (global_label "J1:1" (shape bidirectional) (at 125.73 67.31 90) (fields_autoplaced)
     (effects (font (size 1.1 1.1)) (justify left))
@@
         )
       )
-      (project "LitexCNC-7c81"
+      (project "LITEXCNC-HUB75HAT"
         (path "/d03ad006-987f-4980-aa86-8f7e7030b027/ddedc954-987e-49a5-be4a-196a3f503e33"
           (reference "J10") (unit 1)
@@
         )
       )
-      (project "LitexCNC-7c81"
+      (project "LITEXCNC-HUB75HAT"
         (path "/d03ad006-987f-4980-aa86-8f7e7030b027/ddedc954-987e-49a5-be4a-196a3f503e33"
           (reference "#FLG01") (unit 1)
@@
         )
       )
-      (project "LitexCNC-7c81"
+      (project "LITEXCNC-HUB75HAT"
         (path "/d03ad006-987f-4980-aa86-8f7e7030b027/ddedc954-987e-49a5-be4a-196a3f503e33"
           (reference "#PWR049") (unit 1)
@@
         )
       )
-      (project "LitexCNC-7c81"
+      (project "LITEXCNC-HUB75HAT"
         (path "/d03ad006-987f-4980-aa86-8f7e7030b027/ddedc954-987e-49a5-be4a-196a3f503e33"
           (reference "#PWR034") (unit 1)
@@
         )
       )
-      (project "LitexCNC-7c81"
+      (project "LITEXCNC-HUB75HAT"
         (path "/d03ad006-987f-4980-aa86-8f7e7030b027/ddedc954-987e-49a5-be4a-196a3f503e33"
           (reference "#PWR050") (unit 1)
@@
         )
       )
-      (project "LitexCNC-7c81"
+      (project "LITEXCNC-HUB75HAT"
         (path "/d03ad006-987f-4980-aa86-8f7e7030b027/ddedc954-987e-49a5-be4a-196a3f503e33"
           (reference "#PWR044") (unit 1)
@@
         )
       )
-      (project "LitexCNC-7c81"
+      (project "LITEXCNC-HUB75HAT"
         (path "/d03ad006-987f-4980-aa86-8f7e7030b027/ddedc954-987e-49a5-be4a-196a3f503e33"
           (reference "#PWR036") (unit 1)
@@
         )
       )
-      (project "LitexCNC-7c81"
+      (project "LITEXCNC-HUB75HAT"
         (path "/d03ad006-987f-4980-aa86-8f7e7030b027/ddedc954-987e-49a5-be4a-196a3f503e33"
           (reference "J16") (unit 1)
@@
         )
       )
-      (project "LitexCNC-7c81"
+      (project "LITEXCNC-HUB75HAT"
         (path "/d03ad006-987f-4980-aa86-8f7e7030b027/ddedc954-987e-49a5-be4a-196a3f503e33"
           (reference "C8") (unit 1)
@@
         )
       )
-      (project "LitexCNC-7c81"
+      (project "LITEXCNC-HUB75HAT"
         (path "/d03ad006-987f-4980-aa86-8f7e7030b027/ddedc954-987e-49a5-be4a-196a3f503e33"
           (reference "#PWR038") (unit 1)
@@
         )
       )
-      (project "LitexCNC-7c81"
+      (project "LITEXCNC-HUB75HAT"
         (path "/d03ad006-987f-4980-aa86-8f7e7030b027/ddedc954-987e-49a5-be4a-196a3f503e33"
           (reference "J12") (unit 1)
@@
         )
       )
-      (project "LitexCNC-7c81"
+      (project "LITEXCNC-HUB75HAT"
         (path "/d03ad006-987f-4980-aa86-8f7e7030b027/ddedc954-987e-49a5-be4a-196a3f503e33"
           (reference "#PWR043") (unit 1)
@@
         )
       )
-      (project "LitexCNC-7c81"
+      (project "LITEXCNC-HUB75HAT"
         (path "/d03ad006-987f-4980-aa86-8f7e7030b027/ddedc954-987e-49a5-be4a-196a3f503e33"
           (reference "#PWR047") (unit 1)
@@
         )
       )
-      (project "LitexCNC-7c81"
+      (project "LITEXCNC-HUB75HAT"
         (path "/d03ad006-987f-4980-aa86-8f7e7030b027/ddedc954-987e-49a5-be4a-196a3f503e33"
           (reference "#PWR048") (unit 1)
@@
         )
       )
-      (project "LitexCNC-7c81"
+      (project "LITEXCNC-HUB75HAT"
         (path "/d03ad006-987f-4980-aa86-8f7e7030b027/ddedc954-987e-49a5-be4a-196a3f503e33"
           (reference "#PWR046") (unit 1)
@@
         )
       )
-      (project "LitexCNC-7c81"
+      (project "LITEXCNC-HUB75HAT"
         (path "/d03ad006-987f-4980-aa86-8f7e7030b027/ddedc954-987e-49a5-be4a-196a3f503e33"
           (reference "#PWR051") (unit 1)
@@
         )
       )
-      (project "LitexCNC-7c81"
+      (project "LITEXCNC-HUB75HAT"
         (path "/d03ad006-987f-4980-aa86-8f7e7030b027/ddedc954-987e-49a5-be4a-196a3f503e33"
           (reference "J5") (unit 1)
@@
         )
       )
-      (project "LitexCNC-7c81"
+      (project "LITEXCNC-HUB75HAT"
         (path "/d03ad006-987f-4980-aa86-8f7e7030b027/ddedc954-987e-49a5-be4a-196a3f503e33"
           (reference "C7") (unit 1)
@@
         )
       )
-      (project "LitexCNC-7c81"
+      (project "LITEXCNC-HUB75HAT"
         (path "/d03ad006-987f-4980-aa86-8f7e7030b027/ddedc954-987e-49a5-be4a-196a3f503e33"
           (reference "#PWR035") (unit 1)
@@
         )
       )
-      (project "LitexCNC-7c81"
+      (project "LITEXCNC-HUB75HAT"
         (path "/d03ad006-987f-4980-aa86-8f7e7030b027/ddedc954-987e-49a5-be4a-196a3f503e33"
           (reference "J15") (unit 1)
@@
         )
       )
-      (project "LitexCNC-7c81"
+      (project "LITEXCNC-HUB75HAT"
         (path "/d03ad006-987f-4980-aa86-8f7e7030b027/ddedc954-987e-49a5-be4a-196a3f503e33"
           (reference "#PWR040") (unit 1)
@@
         )
       )
-      (project "LitexCNC-7c81"
+      (project "LITEXCNC-HUB75HAT"
         (path "/d03ad006-987f-4980-aa86-8f7e7030b027/ddedc954-987e-49a5-be4a-196a3f503e33"
           (reference "#PWR053") (unit 1)
@@
         )
       )
-      (project "LitexCNC-7c81"
+      (project "LITEXCNC-HUB75HAT"
         (path "/d03ad006-987f-4980-aa86-8f7e7030b027/ddedc954-987e-49a5-be4a-196a3f503e33"
           (reference "J11") (unit 1)
@@
         )
       )
-      (project "LitexCNC-7c81"
+      (project "LITEXCNC-HUB75HAT"
         (path "/d03ad006-987f-4980-aa86-8f7e7030b027/ddedc954-987e-49a5-be4a-196a3f503e33"
           (reference "#PWR039") (unit 1)
@@
         )
       )
-      (project "LitexCNC-7c81"
+      (project "LITEXCNC-HUB75HAT"
         (path "/d03ad006-987f-4980-aa86-8f7e7030b027/ddedc954-987e-49a5-be4a-196a3f503e33"
           (reference "J14") (unit 1)
@@
         )
       )
-      (project "LitexCNC-7c81"
+      (project "LITEXCNC-HUB75HAT"
         (path "/d03ad006-987f-4980-aa86-8f7e7030b027/ddedc954-987e-49a5-be4a-196a3f503e33"
           (reference "#PWR042") (unit 1)
@@
         )
       )
-      (project "LitexCNC-7c81"
+      (project "LITEXCNC-HUB75HAT"
         (path "/d03ad006-987f-4980-aa86-8f7e7030b027/ddedc954-987e-49a5-be4a-196a3f503e33"
           (reference "J13") (unit 1)
@@
         )
       )
-      (project "LitexCNC-7c81"
+      (project "LITEXCNC-HUB75HAT"
         (path "/d03ad006-987f-4980-aa86-8f7e7030b027/ddedc954-987e-49a5-be4a-196a3f503e33"
           (reference "#PWR041") (unit 1)
@@
         )
       )
-      (project "LitexCNC-7c81"
+      (project "LITEXCNC-HUB75HAT"
         (path "/d03ad006-987f-4980-aa86-8f7e7030b027/ddedc954-987e-49a5-be4a-196a3f503e33"
           (reference "J4") (unit 1)
@@
         )
       )
-      (project "LitexCNC-7c81"
+      (project "LITEXCNC-HUB75HAT"
         (path "/d03ad006-987f-4980-aa86-8f7e7030b027/ddedc954-987e-49a5-be4a-196a3f503e33"
           (reference "J6") (unit 1)
@@
         )
       )
-      (project "LitexCNC-7c81"
+      (project "LITEXCNC-HUB75HAT"
         (path "/d03ad006-987f-4980-aa86-8f7e7030b027/ddedc954-987e-49a5-be4a-196a3f503e33"
           (reference "#PWR045") (unit 1)
@@
         )
       )
-      (project "LitexCNC-7c81"
+      (project "LITEXCNC-HUB75HAT"
         (path "/d03ad006-987f-4980-aa86-8f7e7030b027/ddedc954-987e-49a5-be4a-196a3f503e33"
           (reference "#PWR037") (unit 1)
@@
         )
       )
-      (project "LitexCNC-7c81"
+      (project "LITEXCNC-HUB75HAT"
         (path "/d03ad006-987f-4980-aa86-8f7e7030b027/ddedc954-987e-49a5-be4a-196a3f503e33"
           (reference "#PWR052") (unit 1)
@@
         )
       )
-      (project "LitexCNC-7c81"
+      (project "LITEXCNC-HUB75HAT"
         (path "/d03ad006-987f-4980-aa86-8f7e7030b027/ddedc954-987e-49a5-be4a-196a3f503e33"
           (reference "J9") (unit 1)

Commit message: Proto-type board finished
Connections:
- net J4:9: now reaches J23.10 (Pin_10)
- net ENA: now reaches J23.11 (Pin_11)
- net SPI_CS: now reaches J23.12 (Pin_12)
- net J4:7: now reaches J23.8 (Pin_8)
- net J4:8: now reaches J23.9 (Pin_9)
Changed lines of the file:
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@@
+    )
+  )
+  (global_label "J4:8" (shape bidirectional) (at 44.45 80.01 270) (fields_autoplaced)
+    (effects (font (size 1.1 1.1)) (justify right))
+    (property "Intersheetrefs" "${INTERSHEET_REFS}" (at 44.45 87.0149 90)
+      (effects (font (size 1.27 1.27)) (justify right) hide)
     )
   )
@@
     (property "Intersheetrefs" "${INTERSHEET_REFS}" (at 113.03 48.9149 90)
       (effects (font (size 1.27 1.27)) (justify right) hide)
+    )
+  )
+  (global_label "SPI_CS" (shape input) (at 46.99 67.31 90) (fields_autoplaced)
+    (effects (font (size 1 1)) (justify left))
+    (property "Intersheetrefs" "${INTERSHEET_REFS}" (at 46.99 59.8168 90)
+      (effects (font (size 1.27 1.27)) (justify left) hide)
     )
   )
@@
     )
   )
+  (global_label "J4:7" (shape bidirectional) (at 41.91 67.31 90) (fields_autoplaced)
+    (effects (font (size 1.1 1.1)) (justify left))
+    (property "Intersheetrefs" "${INTERSHEET_REFS}" (at 41.91 60.3051 90)
+      (effects (font (size 1.27 1.27)) (justify left) hide)
+    )
+  )
   (global_label "J4:4" (shape bidirectional) (at 39.37 80.01 270) (fields_autoplaced)
     (effects (font (size 1.1 1.1)) (justify right))
@@
     )
   )
+  (global_label "ENA" (shape output) (at 46.99 80.01 270) (fields_autoplaced)
+    (effects (font (size 1 1)) (justify right))
+    (property "Intersheetrefs" "${INTERSHEET_REFS}" (at 46.99 85.1698 90)
+      (effects (font (size 1.27 1.27)) (justify right) hide)
+    )
+  )
   (global_label "J2:4" (shape bidirectional) (at 100.33 80.01 270) (fields_autoplaced)
     (effects (font (size 1.1 1.1)) (justify right))
@@
     )
   )
+  (global_label "J4:9" (shape bidirectional) (at 44.45 67.31 90) (fields_autoplaced)
+    (effects (font (size 1.1 1.1)) (justify left))
+    (property "Intersheetrefs" "${INTERSHEET_REFS}" (at 44.45 60.3051 90)
+      (effects (font (size 1.27 1.27)) (justify left) hide)
+    )
+  )

Commit message: Version 1.1
Parts:
- removed C8: 1u, Capacitor_SMD:C_1206_3216Metric_Pad1.33x1.80mm_HandSolder, symbol Device:C
- removed C9: 100n, Capacitor_SMD:C_1206_3216Metric_Pad1.33x1.80mm_HandSolder, symbol Device:C
Connections:
- net ENA renamed ENA_IN
- net VDD: no longer names the net of J21.2 (Pin_2)
- net VDD: no longer J20.2 (Pin_2)
Changed lines of the file:
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@@
 (kicad_sch (version 20230121) (generator eeschema)
   (paper "A4")
-  (junction (at 135.89 105.41) (diameter 0) (color 0 0 0 0)
-  )
-  (junction (at 125.73 118.11) (diameter 0) (color 0 0 0 0)
-  )
-  (junction (at 120.65 105.41) (diameter 0) (color 0 0 0 0)
-  )
-  (junction (at 125.73 105.41) (diameter 0) (color 0 0 0 0)
-  )
-  (junction (at 135.89 118.11) (diameter 0) (color 0 0 0 0)
-  )
   (junction (at 120.65 118.11) (diameter 0) (color 0 0 0 0)
   )
@@
   )
   (wire (pts (xy 92.71 107.95) (xy 91.44 107.95))
-    (stroke (width 0) (type solid))
-  )
-  (wire (pts (xy 135.89 105.41) (xy 137.16 105.41))
     (stroke (width 0) (type solid))
   )
@@
     (stroke (width 0) (type solid))
   )
-  (wire (pts (xy 135.89 105.41) (xy 135.89 107.95))
-    (stroke (width 0) (type solid))
-  )
-  (wire (pts (xy 120.65 105.41) (xy 125.73 105.41))
-    (stroke (width 0) (type solid))
-  )
   (wire (pts (xy 82.55 67.31) (xy 82.55 62.23))
     (stroke (width 0) (type solid))
@@
     (stroke (width 0) (type solid))
   )
-  (wire (pts (xy 110.49 105.41) (xy 120.65 105.41))
-    (stroke (width 0) (type solid))
-  )
   (wire (pts (xy 36.83 67.31) (xy 36.83 64.77))
     (stroke (width 0) (type solid))
@@
     (stroke (width 0) (type dash))
   )
-  (wire (pts (xy 125.73 105.41) (xy 135.89 105.41))
-    (stroke (width 0) (type solid))
-  )
   (polyline (pts (xy 97.79 97.79) (xy 97.79 125.73))
     (stroke (width 0) (type dash))
@@
     (stroke (width 0) (type solid))
   )
-  (wire (pts (xy 125.73 118.11) (xy 120.65 118.11))
-    (stroke (width 0) (type solid))
-  )
-  (wire (pts (xy 135.89 104.14) (xy 135.89 105.41))
+  (wire (pts (xy 120.65 118.11) (xy 135.89 118.11))
     (stroke (width 0) (type solid))
   )
@@
   (polyline (pts (xy 24.13 21.59) (xy 24.13 95.25))
     (stroke (width 0) (type dash))
-  )
-  (wire (pts (xy 110.49 110.49) (xy 110.49 105.41))
-    (stroke (width 0) (type solid))
-  )
-  (wire (pts (xy 135.89 118.11) (xy 125.73 118.11))
-    (stroke (width 0) (type solid))
-  )
-  (wire (pts (xy 125.73 115.57) (xy 125.73 118.11))
-    (stroke (width 0) (type solid))
   )
   (wire (pts (xy 128.27 64.77) (xy 128.27 67.31))
@@
     (stroke (width 0) (type dash))
   )
-  (wire (pts (xy 125.73 105.41) (xy 125.73 107.95))
-    (stroke (width 0) (type solid))
-  )
   (wire (pts (xy 52.07 67.31) (xy 52.07 64.77))
     (stroke (width 0) (type solid))
@@
     (stroke (width 0) (type solid))
   )
-  (wire (pts (xy 120.65 105.41) (xy 120.65 110.49))
-    (stroke (width 0) (type default))
-  )
   (polyline (pts (xy 153.67 95.25) (xy 153.67 21.59))
     (stroke (width 0) (type dash))
-  )
-  (wire (pts (xy 135.89 115.57) (xy 135.89 118.11))
-    (stroke (width 0) (type solid))
   )
   (wire (pts (xy 109.22 113.03) (xy 110.49 113.03))
@@
     )
   )
-  (global_label "ENA" (shape output) (at 46.99 80.01 270) (fields_autoplaced)
+  (global_label "ENA_IN" (shape output) (at 46.99 80.01 270) (fields_autoplaced)
     (effects (font (size 1 1)) (justify right))
-    (property "Intersheetrefs" "${INTERSHEET_REFS}" (at 46.99 85.1698 90)
+    (property "Intersheetrefs" "${INTERSHEET_REFS}" (at 46.99 87.4555 90)
       (effects (font (size 1.27 1.27)) (justify right) hide)
     )
@@
     )
   )
-  (symbol (lib_id "power:PWR_FLAG") (at 137.16 105.41 270) (unit 1)
-    (in_bom yes) (on_board yes) (dnp no) (fields_autoplaced)
-    (property "Reference" "#FLG04" (at 139.065 105.41 0)
-      (effects (font (size 1.27 1.27)) hide)
-    )
-    (property "Value" "PWR_FLAG" (at 140.97 105.4099 90)
-      (effects (font (size 1.27 1.27)) (justify left))
-    )
-    (property "Footprint" "" (at 137.16 105.41 0)
-      (effects (font (size 1.27 1.27)) hide)
-    )
-    (property "Datasheet" "~" (at 137.16 105.41 0)
-      (effects (font (size 1.27 1.27)) hide)
-    )
-    (pin "1")
-    (instances
-      (project "chubby-hat"
-        (path "/4807f255-cede-4a86-b009-c3f93cadbbb8/cd3f7ea5-63a4-40ca-a998-c2430d7cb59c"
-          (reference "#FLG04") (unit 1)
-        )
-      )
-      (project "LITEXCNC-HUB75HAT"
-        (path "/d03ad006-987f-4980-aa86-8f7e7030b027/ddedc954-987e-49a5-be4a-196a3f503e33"
-          (reference "#FLG01") (unit 1)
-        )
-      )
-    )
-  )
   (symbol (lib_id "power:GND") (at 67.31 64.77 180) (unit 1)
     (in_bom yes) (on_board yes) (dnp no) (fields_autoplaced)
@@
         (path "/d03ad006-987f-4980-aa86-8f7e7030b027/ddedc954-987e-49a5-be4a-196a3f503e33"
           (reference "#PWR034") (unit 1)
-        )
-      )
-    )
-  )
-  (symbol (lib_id "power:VDD") (at 135.89 104.14 0) (mirror y) (unit 1)
-    (in_bom yes) (on_board yes) (dnp no) (fields_autoplaced)
-    (property "Reference" "#PWR088" (at 135.89 107.95 0)
-      (effects (font (size 1.27 1.27)) hide)
-    )
-    (property "Value" "VDD" (at 135.89 99.06 0)
-      (effects (font (size 1.27 1.27)))
-    )
-    (property "Footprint" "" (at 135.89 104.14 0)
-      (effects (font (size 1.27 1.27)) hide)
-    )
-    (property "Datasheet" "" (at 135.89 104.14 0)
-      (effects (font (size 1.27 1.27)) hide)
-    )
-    (pin "1")
-    (instances
-      (project "chubby-hat"
-        (path "/4807f255-cede-4a86-b009-c3f93cadbbb8/cd3f7ea5-63a4-40ca-a998-c2430d7cb59c"
-          (reference "#PWR088") (unit 1)
-        )
-      )
-      (project "LITEXCNC-HUB75HAT"
-        (path "/d03ad006-987f-4980-aa86-8f7e7030b027/ddedc954-987e-49a5-be4a-196a3f503e33"
-          (reference "#PWR050") (unit 1)
         )
       )
@@
     )
   )
-  (symbol (lib_id "Device:C") (at 135.89 111.76 0) (mirror x) (unit 1)
-    (in_bom yes) (on_board yes) (dnp no) (fields_autoplaced)
-    (property "Reference" "C9" (at 139.7 110.4899 0)
-      (effects (font (size 1.27 1.27)) (justify left))
-    )
-    (property "Value" "100n" (at 139.7 113.0299 0)
-      (effects (font (size 1.27 1.27)) (justify left))
-    )
-    (property "Footprint" "Capacitor_SMD:C_1206_3216Metric_Pad1.33x1.80mm_HandSolder" (at 136.855 107.95 0)
-      (effects (font (size 1.27 1.27)) hide)
-    )
-    (property "Datasheet" "~" (at 135.89 111.76 0)
-      (effects (font (size 1.27 1.27)) hide)
-    )
-    (pin "1")
-    (pin "2")
-    (instances
-      (project "chubby-hat"
-        (path "/4807f255-cede-4a86-b009-c3f93cadbbb8/cd3f7ea5-63a4-40ca-a998-c2430d7cb59c"
-          (reference "C9") (unit 1)
-        )
-      )
-      (project "LITEXCNC-HUB75HAT"
-        (path "/d03ad006-987f-4980-aa86-8f7e7030b027/ddedc954-987e-49a5-be4a-196a3f503e33"
-          (reference "C8") (unit 1)
-        )
-      )
-    )
-  )
   (symbol (lib_id "power:GND") (at 125.73 46.99 0) (unit 1)
     (in_bom yes) (on_board yes) (dnp no) (fields_autoplaced)
@@
         )
       )
-    )
-  )
-  (symbol (lib_id "Device:C") (at 125.73 111.76 0) (mirror x) (unit 1)
-    (in_bom yes) (on_board yes) (dnp no) (fields_autoplaced)
-    (property "Reference" "C8" (at 129.54 110.4899 0)
-      (effects (font (size 1.27 1.27)) (justify left))
-    )
-    (property "Value" "1u" (at 129.54 113.0299 0)
-      (effects (font (size 1.27 1.27)) (justify left))
-    )
-    (property "Footprint" "Capacitor_SMD:C_1206_3216Metric_Pad1.33x1.80mm_HandSolder" (at 126.695 107.95 0)
-      (effects (font (size 1.27 1.27)) hide)
-    )
-    (property "Datasheet" "~" (at 125.73 111.76 0)
-      (effects (font (size 1.27 1.27)) hide)
-    )
-    (pin "1")
-    (pin "2")
-    (instances
-      (project "chubby-hat"
-        (path "/4807f255-cede-4a86-b009-c3f93cadbbb8/cd3f7ea5-63a4-40ca-a998-c2430d7cb59c"
-          (reference "C8") (unit 1)
-        )
-      )
-      (project "LITEXCNC-HUB75HAT"
-        (path "/d03ad006-987f-4980-aa86-8f7e7030b027/ddedc954-987e-49a5-be4a-196a3f503e33"
-          (reference "C7") (unit 1)
-        )
-      )
