File: src/BOB4AXIS/KICAD/BOB4AXIS.kicad_sch (KiCad schematic)
At the start: 47 parts, among them J1 Conn_02x13_Odd_Even, J1 Screw_Terminal_01x03, J2 Screw_Terminal_01x03, J3 Screw_Terminal_01x03, J4 Screw_Terminal_01x03, J5 Screw_Terminal_01x08, J6 Screw_Terminal_01x08, J7 Screw_Terminal_01x08, J8 Screw_Terminal_01x08, U1 LTV-814, U2 LTV-814, U3 LTV-814, U4 LTV-814, U5 AM26LS31CD, U6 AM26LS31CD, U7 KF142V-5_08-2P, U8 74HC86, U9 AM26LS31CD

Commit message: Add pull-down resistor on ENA
Parts:
- C1, C2, C3, C4: LCSC (none) -> C24497
- U5, U6, U9: LCSC (none) -> C6179
- U8: LCSC (none) -> C6763
Changed lines of the file:
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@@
+      (effects (font (size 1.27 1.27)) hide)
+    )
+    (property "LCSC" "C24497" (at 104.14 175.26 0)
       (effects (font (size 1.27 1.27)) hide)
     )
@@
       (effects (font (size 1.27 1.27)) hide)
     )
+    (property "LCSC" "C24497" (at 116.84 175.26 0)
+      (effects (font (size 1.27 1.27)) hide)
+    )
     (pin "1")
     (pin "2")
@@
     )
     (property "Datasheet" "http://www.ti.com/lit/gpn/sn74HC86" (at 43.18 69.85 0)
+      (effects (font (size 1.27 1.27)) hide)
+    )
+    (property "LCSC" "C6763" (at 43.18 69.85 0)
       (effects (font (size 1.27 1.27)) hide)
     )
@@
       (effects (font (size 1.27 1.27)) hide)
     )
+    (property "LCSC" "C24497" (at 78.74 175.26 0)
+      (effects (font (size 1.27 1.27)) hide)
+    )
     (pin "1")
     (pin "2")
@@
       (effects (font (size 1.27 1.27)) hide)
     )
+    (property "LCSC" "C24497" (at 91.44 175.26 0)
+      (effects (font (size 1.27 1.27)) hide)
+    )
     (pin "1")
     (pin "2")
@@
     )
     (property "Datasheet" "https://www.ti.com/lit/ds/symlink/am26ls31.pdf" (at 36.83 133.35 0)
+      (effects (font (size 1.27 1.27)) hide)
+    )
+    (property "LCSC" "C6179" (at 36.83 123.19 0)
       (effects (font (size 1.27 1.27)) hide)
     )
@@
     )
     (property "Datasheet" "http://www.ti.com/lit/gpn/sn74HC86" (at 161.29 69.85 0)
+      (effects (font (size 1.27 1.27)) hide)
+    )
+    (property "LCSC" "C6763" (at 161.29 69.85 0)
       (effects (font (size 1.27 1.27)) hide)
     )
@@
       (effects (font (size 1.27 1.27)) hide)
     )
+    (property "LCSC" "C6763" (at 121.92 69.85 0)
+      (effects (font (size 1.27 1.27)) hide)
+    )
     (pin "1")
     (pin "2")
@@
       (effects (font (size 1.27 1.27)) hide)
     )
+    (property "LCSC" "C6179" (at 124.46 123.19 0)
+      (effects (font (size 1.27 1.27)) hide)
+    )
     (pin "1")
     (pin "10")
@@
     )
     (property "Datasheet" "http://www.ti.com/lit/gpn/sn74HC86" (at 82.55 69.85 0)
+      (effects (font (size 1.27 1.27)) hide)
+    )
+    (property "LCSC" "C6763" (at 82.55 69.85 0)
       (effects (font (size 1.27 1.27)) hide)
     )
@@
       (effects (font (size 1.27 1.27)) hide)
     )
+    (property "LCSC" "C6179" (at 81.28 123.19 0)
+      (effects (font (size 1.27 1.27)) hide)
+    )
     (pin "1")
     (pin "10")
@@
       (effects (font (size 1.27 1.27)) hide)
     )
+    (property "LCSC" "C6763" (at 187.96 71.12 0)
+      (effects (font (size 1.27 1.27)) hide)
+    )
