File: src/BOB4ENCODER/KICAD/BOB4ENCODER.kicad_pcb (KiCad board)
At the start: 2 copper layers, 65 x 93 mm, 34 parts, among them J1 Conn_02x13_Odd_Even, J2 Screw_Terminal_01x08, J3 Screw_Terminal_01x08, J4 Screw_Terminal_01x08, J5 Screw_Terminal_01x08, J6 Conn_02x04_Odd_Even, J7 Conn_02x04_Odd_Even, U1 AM26LV32xD, U2 AM26LV32xD, U3 AM26LV32xD

Commit message: Update latest version
Parts:
- added G***: LOGO, LOGO, F.Cu at (2.59, 78.7)
- added G***: LOGO, LOGO, B.Cu at (59.6, 37.4)
- moved G*** 14.9 mm to (3.00, 38.3)
- moved F1 8.52 mm to (49.1, 14.5)
- moved J6 2.68 mm to (59.0, 13.8)
- moved J7 2.67 mm to (5.95, 10.0)
Connections:
- J6 pad 1: EXT4 -> EXT1
- J6 pad 2: +5V -> ENA
- J6 pad 3: EXT3 -> EXT2
- J6 pad 5: EXT2 -> EXT3
- J6 pad 7: EXT1 -> EXT4
- J6 pad 8: ENA -> +5V
Routing:
- net +5V: track 228.5 -> 220.4 mm
- net EXT4: track 68.2 -> 60.9 mm, vias 0 -> 1
- net EXT3: track 68.2 -> 62.8 mm, vias 0 -> 1
- net EXT2: track 68.2 -> 65.3 mm, vias 0 -> 1
- net ENA: track 191.2 -> 192.6 mm
- net EXT1: track 67.4 -> 66.1 mm, vias 0 -> 1
- net 5V_Fused: track 57.6 -> 58.6 mm
- net ENC1_A-: track 97.6 -> 97.3 mm, vias 1 -> 0
- net GND: vias 52 -> 51
Other:
- board text added: "5V ENCODERS ONLY!"
- board text added: "JLCJLCJLCJLC"
- board text added: "REQUIRED HUB75HAT SETTINGS: - breakout power ENABLED - pull-up / down NOT REQUIRED"
- board text added: "SERIAL"
