File: src/BOB4ENCODER/KICAD/BOB4ENCODER.kicad_sch (KiCad schematic)
At the start: 32 parts, among them J1 Conn_02x13_Odd_Even, J2 Screw_Terminal_01x08, J3 Screw_Terminal_01x08, J4 Screw_Terminal_01x08, J5 Screw_Terminal_01x08, J6 Conn_02x04_Odd_Even, J7 Conn_02x04_Odd_Even, U1 AM26LV32xD, U2 AM26LV32xD, U3 AM26LV32xD

Commit message: Update latest version
Connections:
- net +5V: now also J6.8 (Pin_8); no longer J6.2 (Pin_2)
- net ENA: now also J6.2 (Pin_2); no longer J6.8 (Pin_8)
- net EXT1: now also J6.1 (Pin_1); no longer J6.7 (Pin_7)
- net EXT2: now also J6.3 (Pin_3); no longer J6.5 (Pin_5)
- net EXT3: now also J6.5 (Pin_5); no longer J6.3 (Pin_3)
- net EXT4: now also J6.7 (Pin_7); no longer J6.1 (Pin_1)
Changed lines of the file:
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@@
-    )
-  )
-  (global_label "EXT1" (shape bidirectional) (at 204.47 57.15 180) (fields_autoplaced)
-    (effects (font (size 1.1 1.1)) (justify right))
-    (property "Intersheetrefs" "${INTERSHEET_REFS}" (at 196.9937 57.15 0)
-      (effects (font (size 1.27 1.27)) (justify right) hide)
     )
   )
@@
     (effects (font (size 1 1)) (justify right))
     (property "Intersheetrefs" "${INTERSHEET_REFS}" (at 27.7178 101.6 0)
+      (effects (font (size 1.27 1.27)) (justify right) hide)
+    )
+  )
+  (global_label "EXT1" (shape bidirectional) (at 204.47 49.53 180) (fields_autoplaced)
+    (effects (font (size 1.1 1.1)) (justify right))
+    (property "Intersheetrefs" "${INTERSHEET_REFS}" (at 196.9937 49.53 0)
       (effects (font (size 1.27 1.27)) (justify right) hide)
     )
@@
     )
   )
+  (global_label "EXT2" (shape bidirectional) (at 204.47 52.07 180) (fields_autoplaced)
+    (effects (font (size 1.1 1.1)) (justify right))
+    (property "Intersheetrefs" "${INTERSHEET_REFS}" (at 196.9937 52.07 0)
+      (effects (font (size 1.27 1.27)) (justify right) hide)
+    )
+  )
   (global_label "5V_Fused" (shape input) (at 254 114.3 180) (fields_autoplaced)
     (effects (font (size 1 1)) (justify right))
@@
     )
   )
+  (global_label "EXT3" (shape bidirectional) (at 204.47 54.61 180) (fields_autoplaced)
+    (effects (font (size 1.1 1.1)) (justify right))
+    (property "Intersheetrefs" "${INTERSHEET_REFS}" (at 196.9937 54.61 0)
+      (effects (font (size 1.27 1.27)) (justify right) hide)
+    )
+  )
   (global_label "ENC2_Z-" (shape input) (at 135.89 107.95 180) (fields_autoplaced)
     (effects (font (size 1 1)) (justify right))
@@
     (effects (font (size 1 1)) (justify right))
     (property "Intersheetrefs" "${INTERSHEET_REFS}" (at 244.7925 109.22 0)
+      (effects (font (size 1.27 1.27)) (justify right) hide)
+    )
+  )
+  (global_label "EXT4" (shape bidirectional) (at 204.47 57.15 180) (fields_autoplaced)
+    (effects (font (size 1.1 1.1)) (justify right))
+    (property "Intersheetrefs" "${INTERSHEET_REFS}" (at 196.9937 57.15 0)
       (effects (font (size 1.27 1.27)) (justify right) hide)
     )
@@
     )
   )
+  (global_label "ENA" (shape input) (at 217.17 49.53 0) (fields_autoplaced)
+    (effects (font (size 1.1 1.1)) (justify left))
+    (property "Intersheetrefs" "${INTERSHEET_REFS}" (at 222.8458 49.53 0)
+      (effects (font (size 1.27 1.27)) (justify left) hide)
+    )
+  )
   (global_label "ENC4_A" (shape input) (at 252.73 55.88 180) (fields_autoplaced)
     (effects (font (size 1.1 1.1)) (justify right))
@@
     )
   )
-  (global_label "EXT4" (shape bidirectional) (at 204.47 49.53 180) (fields_autoplaced)
-    (effects (font (size 1.1 1.1)) (justify right))
-    (property "Intersheetrefs" "${INTERSHEET_REFS}" (at 196.9937 49.53 0)
-      (effects (font (size 1.27 1.27)) (justify right) hide)
-    )
-  )
   (global_label "ENC1_A+" (shape input) (at 214.63 99.06 180) (fields_autoplaced)
     (effects (font (size 1 1)) (justify right))
@@
     )
   )
-  (global_label "ENA" (shape input) (at 217.17 57.15 0) (fields_autoplaced)
-    (effects (font (size 1.1 1.1)) (justify left))
-    (property "Intersheetrefs" "${INTERSHEET_REFS}" (at 222.8458 57.15 0)
-      (effects (font (size 1.27 1.27)) (justify left) hide)
-    )
-  )
   (global_label "5V_Fused" (shape input) (at 254 149.86 180) (fields_autoplaced)
     (effects (font (size 1 1)) (justify right))
@@
     (effects (font (size 1 1)) (justify right))
     (property "Intersheetrefs" "${INTERSHEET_REFS}" (at 244.8878 96.52 0)
-      (effects (font (size 1.27 1.27)) (justify right) hide)
-    )
-  )
-  (global_label "EXT2" (shape bidirectional) (at 204.47 54.61 180) (fields_autoplaced)
-    (effects (font (size 1.1 1.1)) (justify right))
-    (property "Intersheetrefs" "${INTERSHEET_REFS}" (at 196.9937 54.61 0)
       (effects (font (size 1.27 1.27)) (justify right) hide)
     )
@@
     (effects (font (size 1 1)) (justify right))
     (property "Intersheetrefs" "${INTERSHEET_REFS}" (at 244.7449 104.14 0)
-      (effects (font (size 1.27 1.27)) (justify right) hide)
-    )
-  )
-  (global_label "EXT3" (shape bidirectional) (at 204.47 52.07 180) (fields_autoplaced)
-    (effects (font (size 1.1 1.1)) (justify right))
-    (property "Intersheetrefs" "${INTERSHEET_REFS}" (at 196.9937 52.07 0)
       (effects (font (size 1.27 1.27)) (justify right) hide)
     )
@@
         (path "/9693837c-ee26-4f84-93b4-ccfecde69efc"
           (reference "JP11") (unit 1)
-        )
-      )
-    )
-  )
-  (symbol (lib_id "power:+5V") (at 217.17 49.53 270) (unit 1)
-    (in_bom yes) (on_board yes) (dnp no) (fields_autoplaced)
-    (property "Reference" "#PWR029" (at 213.36 49.53 0)
-      (effects (font (size 1.27 1.27)) hide)
-    )
-    (property "Value" "+5V" (at 220.98 49.53 90)
-      (effects (font (size 1.27 1.27)) (justify left))
-    )
-    (property "Footprint" "" (at 217.17 49.53 0)
-      (effects (font (size 1.27 1.27)) hide)
-    )
-    (property "Datasheet" "" (at 217.17 49.53 0)
-      (effects (font (size 1.27 1.27)) hide)
-    )
-    (pin "1")
-    (instances
-      (project "BOB4ENCODER"
-        (path "/9693837c-ee26-4f84-93b4-ccfecde69efc"
-          (reference "#PWR029") (unit 1)
-        )
-      )
-      (project "BOB4AXIS"
-        (path "/daea1869-e1ef-4a14-b8f5-612be4c11ee9"
-          (reference "#PWR053") (unit 1)
         )
       )
@@
         )
       )
+    )
+  )
+  (symbol (lib_id "power:+5V") (at 217.17 57.15 270) (unit 1)
+    (in_bom yes) (on_board yes) (dnp no) (fields_autoplaced)
+    (property "Reference" "#PWR029" (at 213.36 57.15 0)
+      (effects (font (size 1.27 1.27)) hide)
+    )
+    (property "Value" "+5V" (at 220.98 57.15 90)
+      (effects (font (size 1.27 1.27)) (justify left))
+    )
+    (property "Footprint" "" (at 217.17 57.15 0)
+      (effects (font (size 1.27 1.27)) hide)
+    )
+    (property "Datasheet" "" (at 217.17 57.15 0)
+      (effects (font (size 1.27 1.27)) hide)
+    )
+    (pin "1")
+    (instances
+      (project "BOB4ENCODER"
+        (path "/9693837c-ee26-4f84-93b4-ccfecde69efc"
+          (reference "#PWR029") (unit 1)
+        )
+      )
+      (project "BOB4AXIS"
+        (path "/daea1869-e1ef-4a14-b8f5-612be4c11ee9"
+          (reference "#PWR053") (unit 1)
+        )
+      )
